File: projects/main-board/esp32.kicad_sch (KiCad schematic)
At the start: 21 parts, among them J6 Conn_01x06, Y1 ABM10W-40.0000MHZ-8-B1U-T3

Commit message: Updated schematics with new symbols
Parts:
- removed J8: ~, symbol symbol-library:USB4105-GF-A
- removed U8: ~, symbol symbol-library:ESP32-C6FH4
- removed Y1: ABM10W-40.0000MHZ-8-B1U-T3, symbol symbol-library:ABM10W-40.0000MHZ-8-B1U-T3
- added J1: USB4105-GF-A, footprint-library:USB4105-GF-A, symbol symbol-library:USB4105-GF-A
- added U5: ESP32-C6FH4, footprint-library:ESP32-C6FH4, symbol symbol-library:ESP32-C6FH4
- added Y2: ABM10W-40.0000MHZ-8-B1U-T3, footprint-library:XTAL_ABM10W-40.0000MHZ-8-B1U-T3, symbol symbol-library:ABM10W-40.0000MHZ-8-B1U-T3
Connections:
- net 3V3: now also U5.29 (VDDA1), U5.32 (VDDA2)
- net DEBUG_UART.RX: now also U5.24 (SDIO_CLK)
- net DEBUG_UART.TX: now also U5.23 (SDIO_CMD)
- net ESP32_EN: now also U5.4 (CHIP_PU)
- net ESP32_GPIO.2: now also U5.8 (GPIO2)
- net ESP32_GPIO.3: now also U5.9 (GPIO3)
- net ESP32_GPIO.8: now also U5.14 (GPIO8)
- net ESP32_GPIO.9: now also U5.15 (GPIO9)
- net ESP32_UART.RX: now also U5.22 (U0RXD)
- net ESP32_UART.TX: now also U5.21 (U0TXD)
- net GND: now also J1.A1 (GND), J1.A12 (GND), J1.B1 (GND), J1.B12 (GND), J1.SHELL (GND), U5.33 (GND), Y2.2 (GND), Y2.4 (GND)
- net JTAG.MTCK: now also U5.12 (MTCK)
- net JTAG.MTDI: now also U5.11 (MTDI)
- net JTAG.MTDO: now also U5.13 (MTDO)
- net JTAG.MTMS: now also U5.10 (MTMS)
- net USB.DN: now also J1.A7 (Dn1), J1.B7 (Dn2), U5.16 (GPIO12)
- net USB.DP: now also J1.A6 (Dp1), J1.B6 (Dp2), U5.17 (GPIO13)
- net at C82.1, L4.1: now also U5.1 (ANT)
- net at C76.1, C77.1, C78.1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: now also U5.2 (VDDA3P3), U5.3 (VDDA3P3)
- net at C80.1, C81.1: now also U5.20 (VDDPST2), U5.5 (VDDPST1)
- net at C85.1: now also U5.30 (XTAL_N), Y2.3
- net at R10.1: now also U5.31 (XTAL_P)
- net at R60.1: now also J1.A5 (CC1)
- net at R59.1: now also J1.B5 (CC2)
- net at C84.1, R10.2: now also Y2.1

Commit message: Re-annotate schematics.
Parts:
- renumbered C74 to C75, C75 to C76, C76 to C77, C77 to C78, C78 to C79, C79 to C80, C80 to C81, C81 to C82, C84 to C83, C82 to C84, C83 to C85, C85 to C86, J1 to J4, J6 to J5, R60 to R51, R11 to R52, R59 to R53, R10 to R54, U5 to U9, Y2 to Y1
Changed lines of the file:
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@@
 		(dnp no)
 		(fields_autoplaced yes)
-		(property "Reference" "C84"
+		(property "Reference" "C83"
 			(at 201.93 87.6362 0)
 			(effects
@@
 			(project "main-board"
 				(path "/c621b5fd-2ef7-4a67-960d-0ffc72b1245a/9604ec8b-dd8b-4641-a93a-60fcfb624c0c"
-					(reference "C84")
+					(reference "C83")
 					(unit 1)
 				)
@@
 		(dnp no)
 		(fields_autoplaced yes)
-		(property "Reference" "C79"
+		(property "Reference" "C80"
 			(at 93.98 31.7562 0)
 			(effects
@@
 			(project "main-board"
 				(path "/c621b5fd-2ef7-4a67-960d-0ffc72b1245a/9604ec8b-dd8b-4641-a93a-60fcfb624c0c"
-					(reference "C79")
+					(reference "C80")
 					(unit 1)
 				)
@@
 		(dnp no)
 		(fields_autoplaced yes)
-		(property "Reference" "C78"
+		(property "Reference" "C79"
 			(at 81.28 31.7562 0)
 			(effects
@@
 			(project "main-board"
 				(path "/c621b5fd-2ef7-4a67-960d-0ffc72b1245a/9604ec8b-dd8b-4641-a93a-60fcfb624c0c"
-					(reference "C78")
+					(reference "C79")
 					(unit 1)
 				)
@@
 		(dnp no)
 		(fields_autoplaced yes)
-		(property "Reference" "R59"
+		(property "Reference" "R53"
 			(at 58.42 154.9399 0)
 			(effects
@@
 			(project "main-board"
 				(path "/c621b5fd-2ef7-4a67-960d-0ffc72b1245a/9604ec8b-dd8b-4641-a93a-60fcfb624c0c"
-					(reference "R59")
+					(reference "R53")
 					(unit 1)
 				)
@@
 		(dnp no)
 		(fields_autoplaced yes)
-		(property "Reference" "C85"
+		(property "Reference" "C86"
 			(at 240.03 87.6362 0)
 			(effects
@@
 			(project "main-board"
 				(path "/c621b5fd-2ef7-4a67-960d-0ffc72b1245a/9604ec8b-dd8b-4641-a93a-60fcfb624c0c"
-					(reference "C85")
+					(reference "C86")
 					(unit 1)
 				)
@@
 		(dnp no)
 		(fields_autoplaced yes)
-		(property "Reference" "R60"
+		(property "Reference" "R51"
 			(at 49.53 154.9399 0)
 			(effects
@@
 			(project "main-board"
 				(path "/c621b5fd-2ef7-4a67-960d-0ffc72b1245a/9604ec8b-dd8b-4641-a93a-60fcfb624c0c"
-					(reference "R60")
+					(reference "R51")
 					(unit 1)
 				)
@@
 		(dnp no)
 		(fields_autoplaced yes)
-		(property "Reference" "J6"
+		(property "Reference" "J5"
 			(at 138.43 138.4299 0)
 			(effects
@@
 			(project "main-board"
 				(path "/c621b5fd-2ef7-4a67-960d-0ffc72b1245a/9604ec8b-dd8b-4641-a93a-60fcfb624c0c"
-					(reference "J6")
+					(reference "J5")
 					(unit 1)
 				)
@@
 		(on_board yes)
 		(dnp no)
-		(property "Reference" "J1"
+		(property "Reference" "J4"
 			(at 82.296 131.064 0)
 			(effects
@@
 			(project ""
 				(path "/c621b5fd-2ef7-4a67-960d-0ffc72b1245a/9604ec8b-dd8b-4641-a93a-60fcfb624c0c"
-					(reference "J1")
+					(reference "J4")
 					(unit 1)
 				)
@@
 		(dnp no)
 		(fields_autoplaced yes)
-		(property "Reference" "C74"
+		(property "Reference" "C75"
 			(at 31.75 26.6762 0)
 			(effects
@@
 			(project ""
 				(path "/c621b5fd-2ef7-4a67-960d-0ffc72b1245a/9604ec8b-dd8b-4641-a93a-60fcfb624c0c"
-					(reference "C74")
+					(reference "C75")
 					(unit 1)
 				)
@@
 		(dnp no)
 		(fields_autoplaced yes)
-		(property "Reference" "C75"
+		(property "Reference" "C76"
 			(at 43.18 26.6762 0)
 			(effects
@@
 			(project "main-board"
 				(path "/c621b5fd-2ef7-4a67-960d-0ffc72b1245a/9604ec8b-dd8b-4641-a93a-60fcfb624c0c"
-					(reference "C75")
+					(reference "C76")
 					(unit 1)
 				)
@@
 		(dnp no)
 		(fields_autoplaced yes)
-		(property "Reference" "#PWR0158"
+		(property "Reference" "#PWR0120"
 			(at 129.54 135.89 0)
 			(effects
@@
 			(project "main-board"
 				(path "/c621b5fd-2ef7-4a67-960d-0ffc72b1245a/9604ec8b-dd8b-4641-a93a-60fcfb624c0c"
-					(reference "#PWR0158")
+					(reference "#PWR0120")
 					(unit 1)
 				)
@@
 		(on_board yes)
 		(dnp no)
-		(property "Reference" "R10"
+		(property "Reference" "R54"
 			(at 189.484 83.058 90)
 			(effects
@@
 			(project ""
 				(path "/c621b5fd-2ef7-4a67-960d-0ffc72b1245a/9604ec8b-dd8b-4641-a93a-60fcfb624c0c"
-					(reference "R10")
+					(reference "R54")
 					(unit 1)
 				)
@@
 		(dnp no)
 		(fields_autoplaced yes)
-		(property "Reference" "#PWR0160"
+		(property "Reference" "#PWR0117"
 			(at 46.99 167.64 0)
 			(effects
@@
 			(project "main-board"
 				(path "/c621b5fd-2ef7-4a67-960d-0ffc72b1245a/9604ec8b-dd8b-4641-a93a-60fcfb624c0c"
-					(reference "#PWR0160")
+					(reference "#PWR0117")
 					(unit 1)
 				)
@@
 		(dnp no)
 		(fields_autoplaced yes)
-		(property "Reference" "#PWR0103"
+		(property "Reference" "#PWR0122"
 			(at 186.69 119.38 0)
 			(effects
@@
 			(project ""
 				(path "/c621b5fd-2ef7-4a67-960d-0ffc72b1245a/9604ec8b-dd8b-4641-a93a-60fcfb624c0c"
-					(reference "#PWR0103")
+					(reference "#PWR0122")
 					(unit 1)
 				)
@@
 		(dnp no)
 		(fields_autoplaced yes)
-		(property "Reference" "C77"
+		(property "Reference" "C78"
 			(at 68.58 31.7562 0)
 			(effects
@@
 			(project "main-board"
 				(path "/c621b5fd-2ef7-4a67-960d-0ffc72b1245a/9604ec8b-dd8b-4641-a93a-60fcfb624c0c"
-					(reference "C77")
+					(reference "C78")
 					(unit 1)
 				)
@@
 		(dnp no)
 		(fields_autoplaced yes)
-		(property "Reference" "C81"
+		(property "Reference" "C82"
 			(at 121.92 36.8362 0)
 			(effects
@@
 			(project "main-board"
 				(path "/c621b5fd-2ef7-4a67-960d-0ffc72b1245a/9604ec8b-dd8b-4641-a93a-60fcfb624c0c"
-					(reference "C81")
+					(reference "C82")
 					(unit 1)
 				)
@@
 		(dnp no)
 		(fields_autoplaced yes)
-		(property "Reference" "C82"
+		(property "Reference" "C84"
 			(at 208.28 26.6762 0)
 			(effects
@@
 			(project "main-board"
 				(path "/c621b5fd-2ef7-4a67-960d-0ffc72b1245a/9604ec8b-dd8b-4641-a93a-60fcfb624c0c"
-					(reference "C82")
+					(reference "C84")
 					(unit 1)
 				)
@@
 		(on_board yes)
 		(dnp no)
-		(property "Reference" "Y2"
+		(property "Reference" "Y1"
 			(at 217.17 76.708 0)
 			(effects
@@
 			(project ""
 				(path "/c621b5fd-2ef7-4a67-960d-0ffc72b1245a/9604ec8b-dd8b-4641-a93a-60fcfb624c0c"
-					(reference "Y2")
+					(reference "Y1")
 					(unit 1)
 				)
@@
 		(dnp no)
 		(fields_autoplaced yes)
-		(property "Reference" "C83"
+		(property "Reference" "C85"
 			(at 226.06 26.6762 0)
 			(effects
@@
 			(project "main-board"
 				(path "/c621b5fd-2ef7-4a67-960d-0ffc72b1245a/9604ec8b-dd8b-4641-a93a-60fcfb624c0c"
-					(reference "C83")
+					(reference "C85")
 					(unit 1)
 				)
@@
 		(dnp no)
 		(fields_autoplaced yes)
-		(property "Reference" "C80"
+		(property "Reference" "C81"
 			(at 107.95 36.8362 0)
 			(effects
@@
 			(project "main-board"
 				(path "/c621b5fd-2ef7-4a67-960d-0ffc72b1245a/9604ec8b-dd8b-4641-a93a-60fcfb624c0c"
-					(reference "C80")
+					(reference "C81")
 					(unit 1)
 				)
@@
 		(dnp no)
 		(fields_autoplaced yes)
-		(property "Reference" "C76"
+		(property "Reference" "C77"
 			(at 55.88 31.7562 0)
 			(effects
@@
 			(project "main-board"
 				(path "/c621b5fd-2ef7-4a67-960d-0ffc72b1245a/9604ec8b-dd8b-4641-a93a-60fcfb624c0c"
-					(reference "C76")
+					(reference "C77")
 					(unit 1)
 				)
@@
 		(dnp no)
 		(fields_autoplaced yes)
-		(property "Reference" "R11"
+		(property "Reference" "R52"
 			(at 57.15 49.5299 0)
 			(effects
@@
 			(project "main-board"
 				(path "/c621b5fd-2ef7-4a67-960d-0ffc72b1245a/9604ec8b-dd8b-4641-a93a-60fcfb624c0c"
-					(reference "R11")
+					(reference "R52")
 					(unit 1)
 				)
@@
 		(on_board yes)
 		(dnp no)
-		(property "Reference" "#PWR0161"
+		(property "Reference" "#PWR0119"
 			(at 105.41 190.5 0)
 			(effects
@@
 			(project "main-board"
 				(path "/c621b5fd-2ef7-4a67-960d-0ffc72b1245a/9604ec8b-dd8b-4641-a93a-60fcfb624c0c"
-					(reference "#PWR0161")
+					(reference "#PWR0119")
 					(unit 1)
 				)
@@
 		(dnp no)
 		(fields_autoplaced yes)
-		(property "Reference" "#PWR0159"
+		(property "Reference" "#PWR0121"
 			(at 129.54 153.67 0)
 			(effects
@@
 			(project "main-board"
 				(path "/c621b5fd-2ef7-4a67-960d-0ffc72b1245a/9604ec8b-dd8b-4641-a93a-60fcfb624c0c"
-					(reference "#PWR0159")
+					(reference "#PWR0121")
 					(unit 1)
 				)
@@
 		(dnp no)
 		(fields_autoplaced yes)
-		(property "Reference" "#PWR0104"
+		(property "Reference" "#PWR0123"
 			(at 220.98 100.33 0)
 			(effects
@@
 			(project "main-board"
 				(path "/c621b5fd-2ef7-4a67-960d-0ffc72b1245a/9604ec8b-dd8b-4641-a93a-60fcfb624c0c"
-					(reference "#PWR0104")
+					(reference "#PWR0123")
 					(unit 1)
 				)
@@
 		(dnp no)
 		(fields_autoplaced yes)
-		(property "Reference" "#PWR0106"
+		(property "Reference" "#PWR0116"
 			(at 29.21 55.88 0)
 			(effects
@@
 			(project "main-board"
 				(path "/c621b5fd-2ef7-4a67-960d-0ffc72b1245a/9604ec8b-dd8b-4641-a93a-60fcfb624c0c"
-					(reference "#PWR0106")
+					(reference "#PWR0116")
 					(unit 1)
 				)
@@
 		(dnp no)
 		(fields_autoplaced yes)
-		(property "Reference" "#PWR0108"
+		(property "Reference" "#PWR0118"
 			(at 54.61 60.96 0)
 			(effects
@@
 			(project "main-board"
 				(path "/c621b5fd-2ef7-4a67-960d-0ffc72b1245a/9604ec8b-dd8b-4641-a93a-60fcfb624c0c"
-					(reference "#PWR0108")
+					(reference "#PWR0118")
 					(unit 1)
 				)
@@
 		(dnp no)
 		(fields_autoplaced yes)
-		(property "Reference" "#PWR0105"
+		(property "Reference" "#PWR0115"
 			(at 29.21 26.67 0)
 			(effects
@@
 			(project "main-board"
 				(path "/c621b5fd-2ef7-4a67-960d-0ffc72b1245a/9604ec8b-dd8b-4641-a93a-60fcfb624c0c"
-					(reference "#PWR0105")
+					(reference "#PWR0115")
 					(unit 1)
 				)
@@
 		(on_board yes)
 		(dnp no)
-		(property "Reference" "U5"
+		(property "Reference" "U9"
 			(at 133.35 20.32 0)
 			(effects
@@
 			(project ""
 				(path "/c621b5fd-2ef7-4a67-960d-0ffc72b1245a/9604ec8b-dd8b-4641-a93a-60fcfb624c0c"
-					(reference "U5")
+					(reference "U9")
 					(unit 1)
 				)
@@
 		(dnp no)
 		(fields_autoplaced yes)
-		(property "Reference" "#PWR0107"
+		(property "Reference" "#PWR0124"
 			(at 223.52 39.37 0)
 			(effects
@@
 			(project "main-board"
 				(path "/c621b5fd-2ef7-4a67-960d-0ffc72b1245a/9604ec8b-dd8b-4641-a93a-60fcfb624c0c"
-					(reference "#PWR0107")
-					(unit 1)
-				)
+					(reference "#PWR0124")
+					(unit 1)
+				)

Commit message: Replace 0.1in header with TC2030
Parts:
- removed J5: Conn_01x06, symbol Connector_Generic:Conn_01x06
- added J2: TC2030, Connector:Tag-Connect_TC2030-IDC-NL_2x03_P1.27mm_Vertical, symbol Connector:TC2030
Connections:
- net DEBUG_UART.RX: now also J2.1
- net DEBUG_UART.TX: now also J2.3
- net ESP32_UART.RX: now also J2.4
- net ESP32_UART.TX: now also J2.2
- net GND: now also J2.5
- no-connect marks 6 -> 7

Commit message: Add capacitor part library.
Parts:
- C75, C78: value 1uF 6.3V -> 1uF 10V
- C77: value 10uF 6.3V -> 10uF 10V
- C79, C80, C81, C82, C84, C85: value 100nF 6.3V -> 100nF 10V
Other:
- moved on the sheet: C80
Changed lines of the file:
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@@
 	)
 	(junction
-		(at 91.44 29.21)
-		(diameter 0)
-		(color 0 0 0 0)
-	)
-	(junction
 		(at 29.21 31.75)
 		(diameter 0)
@@
 	)
 	(junction
+		(at 92.71 29.21)
+		(diameter 0)
+		(color 0 0 0 0)
+	)
+	(junction
 		(at 205.74 24.13)
 		(diameter 0)
@@
 	(wire
 		(pts
-			(xy 128.27 29.21) (xy 91.44 29.21)
+			(xy 128.27 29.21) (xy 92.71 29.21)
 		)
 		(stroke
@@
 	(wire
 		(pts
-			(xy 91.44 36.83) (xy 78.74 36.83)
+			(xy 92.71 36.83) (xy 78.74 36.83)
 		)
 		(stroke
@@
 	(wire
 		(pts
-			(xy 91.44 29.21) (xy 78.74 29.21)
+			(xy 78.74 29.21) (xy 92.71 29.21)
 		)
 		(stroke
@@
 	(wire
 		(pts
-			(xy 91.44 35.56) (xy 91.44 36.83)
+			(xy 92.71 35.56) (xy 92.71 36.83)
 		)
 		(stroke
@@
 	(wire
 		(pts
-			(xy 91.44 29.21) (xy 91.44 30.48)
+			(xy 92.71 29.21) (xy 92.71 30.48)
 		)
 		(stroke
@@
 	(symbol
 		(lib_id "Device:C_Small")
-		(at 91.44 33.02 0)
+		(at 92.71 33.02 0)
 		(unit 1)
 		(exclude_from_sim no)
@@
 		(fields_autoplaced yes)
 		(property "Reference" "C80"
-			(at 93.98 31.7562 0)
+			(at 95.25 31.7562 0)
 			(effects
 				(font
@@
 			)
 		)
-		(property "Value" "100nF 6.3V"
-			(at 93.98 34.2962 0)
+		(property "Value" "100nF 10V"
+			(at 95.25 34.2962 0)
 			(effects
 				(font
@@
 		)
 		(property "Footprint" ""
-			(at 91.44 33.02 0)
+			(at 92.71 33.02 0)
 			(effects
 				(font
@@
 		)
 		(property "Datasheet" "~"
-			(at 91.44 33.02 0)
+			(at 92.71 33.02 0)
 			(effects
 				(font
@@
 		)
 		(property "Description" "Unpolarized capacitor, small symbol"
-			(at 91.44 33.02 0)
+			(at 92.71 33.02 0)
 			(effects
 				(font
@@
 			)
 		)
-		(property "Value" "100nF 6.3V"
+		(property "Value" "100nF 10V"
 			(at 81.28 34.2962 0)
 			(effects
@@
 			)
 		)
-		(property "Value" "1uF 6.3V"
+		(property "Value" "1uF 10V"
 			(at 31.75 29.2162 0)
 			(effects
@@
 			)
 		)
-		(property "Value" "1uF 6.3V"
+		(property "Value" "1uF 10V"
 			(at 68.58 34.2962 0)
 			(effects
@@
 			)
 		)
-		(property "Value" "100nF 6.3V"
+		(property "Value" "100nF 10V"
 			(at 121.92 39.3762 0)
 			(effects
@@
 			)
 		)
-		(property "Value" "100nF 6.3V"
+		(property "Value" "100nF 10V"
 			(at 208.28 29.2162 0)
 			(effects
@@
 			)
 		)
-		(property "Value" "100nF 6.3V"
+		(property "Value" "100nF 10V"
 			(at 226.06 29.2162 0)
 			(effects
@@
 			)
 		)
-		(property "Value" "100nF 6.3V"
+		(property "Value" "100nF 10V"
 			(at 107.95 39.3762 0)
 			(effects
@@
 			)
 		)
-		(property "Value" "10uF 6.3V"
+		(property "Value" "10uF 10V"
 			(at 55.88 34.2962 0)
 			(effects

Commit message: Normalise capacitors
- Add capacitor parts to library.
- Replace all placeholder capacitors
  with the actual part numbers.
Parts:
- removed C75, C78: 1uF 10V, symbol Device:C_Small
- removed C76: 10nF 10V, symbol Device:C_Small
- removed C77: 10uF 10V, symbol Device:C_Small
- removed C79, C80, C81, C82, C84, C85: 100nF 10V, symbol Device:C_Small
- removed C83, C86: 8pF, symbol Device:C_Small
- added C75, C78: 1uF 10V, Capacitor_SMD:C_0402_1005Metric, symbol symbol-library-capacitors:CC0402KRX5R6BB105
- added C76, C79, C80, C81, C82, C84, C85: 100nF 10V, Capacitor_SMD:C_0402_1005Metric, symbol symbol-library-capacitors:CC0402KRX7R6BB104
- added C77: 10uF 10V, Capacitor_SMD:C_0603_1608Metric, symbol symbol-library-capacitors:CC0603MRX5R6BB106
- added C83, C86: 8pF 50V, Capacitor_SMD:C_0402_1005Metric, symbol symbol-library-capacitors:CC0402CRNPO9BN8R0
- renumbered J2 to J5
Connections:
- net 3V3: now also C75.1, C76.1
- net GND: now also C75.2, C76.2, C77.2, C78.2, C79.2, C80.2, C81.2, C82.2, C83.2, C84.2, C85.2, C86.2
- net WIFI_ANT: now also C85.1
- net at R54.2, Y1.1: now also C83.1
- net at U9.2 (VDDA3P3), U9.3 (VDDA3P3): now also C77.1, C78.1, C79.1, C80.1
- net at U9.30 (XTAL_N), Y1.3: now also C86.1
- net at L4.1, U9.1 (ANT): now also C84.1
- net at U9.20 (VDDPST2), U9.5 (VDDPST1): now also C81.1, C82.1
