File: projects/main-board/esp32.kicad_sch (KiCad schematic)
At the start: 21 parts, among them J4 USB4105-GF-A, J5 TC2030, U9 ESP32-C6FH4, Y1 ABM10W-40.0000MHZ-8-B1U-T3

Commit message: Main board PCB layout and routing
- Add 48MHz crystal for STM32
- Add 32kHz crystal for STM32
- Started laying out and routing board
Parts:
- added R63: 0R, Resistor_SMD:R_0402_1005Metric, symbol symbol-library-resistors:RC0402FR-070RL
Connections:
- net 3V3: now also C77.1, C78.1, C79.1, C80.1, C81.1, C82.1, U9.2 (VDDA3P3), U9.20 (VDDPST2), U9.3 (VDDA3P3), U9.5 (VDDPST1)
- net at C86.1, Y1.3: now also R63.2; no longer U9.30 (XTAL_N)
- new net: R63.1, U9.30 (XTAL_N)
- no-connect marks 7 -> 13
Other:
- moved on the sheet: C83, C86, Y1
