File: projects/main-board/pmic.kicad_sch (KiCad schematic)
At the start: 29 parts, among them J3 Conn_01x03, SW1 SW_SPDT

Commit message: Updated schematics with new symbols
Parts:
- removed U14: ~, symbol symbol-library:TPS22992RXPR
- removed U4: ~, symbol symbol-library:MAX77972EWX+T
- removed U6: ~, symbol symbol-library:MPM3805GQB-18-Z
- removed U7: ~, symbol symbol-library:TPSM863253RDXR
- added U16: MPM3805GQB-18-Z, footprint-library:MPM3805GQB-18-Z, symbol symbol-library:MPM3805GQB-18-Z
- added U17: TPSM863253RDXR, footprint-library:TPSM863253RDXR, symbol symbol-library:TPSM863253RDXR
- added U18: TPS22992RXPR, footprint-library:TPS22992RXPR, symbol symbol-library:TPS22992RXPR
- added U3: MAX77972EWX+T, footprint-library:MAX77972EWX+T, symbol symbol-library:MAX77972EWX+T
Connections:
- net 1V8: now also U16.12 (OUT_S), U16.5 (OUT), U16.6 (OUT)
- net 3V3: now also U17.3 (VOUT), U17.7 (VOS)
- net ALRT: now also U3.B4 (ALRT)
- net CC1: now also U3.F3 (CC1)
- net CC2: now also U3.F4 (CC2)
- net CHGEN: now also U3.E3 (CHGEN)
- net DATAMUX: now also U3.B3 (DATAMUX)
- net GND: now also U16.1 (PGND), U16.11 (AGND), U16.2 (PGND), U17.4 (PGND), U18.4 (GND), U3.A6 (GND), U3.B5 (BATTSN), U3.E1 (PGND), U3.E2 (PGND)
- net I2C.SCL: now also U3.B6 (SCL)
- net I2C.SDA: now also U3.C6 (SDA)
- net INOKB: now also U3.C3 (INOKB)
- net STAT: now also U3.A3 (STAT)
- net SYS_PGOOD: now also U16.9 (EN), U17.6 (EN), U18.3 (PG)
- net USB.DN: now also U3.F6 (DN)
- net USB.DP: now also U3.F5 (DP)
- net VBAT: now also U3.C4 (BATTSP/CSN)
- net VBUS: now also U3.B1 (CHGIN), U3.B2 (CHGIN)
- net VSYS: now also U16.7 (VIN), U17.1 (VIN), U18.6 (VOUT)
- net VSYS_IN: now also U18.1 (VBIAS), U18.2 (VIN), U3.E4 (SYS), U3.E5 (SYS), U3.E6 (SYS)
- net at C65.1, C66.1, R9.1: now also U3.C5 (CSP), U3.D4 (BATT), U3.D5 (BATT), U3.D6 (BATT)
- net at R7.1: now also U3.A2 (ICHG)
- net at C62.2, L2.1: now also U3.D1 (LX), U3.D2 (LX), U3.D3 (LX)
- net at C61.1: now also U3.C1 (BYP), U3.C2 (BYP)
- net at C62.1: now also U3.F1 (BST)
- net at R6.2: now also U3.A1 (VCHG)
- net at J3.2 (Pin_2): now also U3.A4 (THM)
- net at C60.1: now also U3.A5 (VDD)
- net at C67.1: now also U3.F2 (PVL)
- net at R48.2: now also U18.5 (QOD)
- net at SW1.1 (A): now also U18.8 (ON)
- net at C107.1: now also U18.7 (CT)

Commit message: Re-annotate schematics.
Parts:
- renumbered C68 to C59, C107 to C60, C69 to C61, C70 to C62, C71 to C63, C60 to C64, C72 to C65, C73 to C66, C62 to C67, C63 to C68, C67 to C69, C65 to C70, C64 to C71, C61 to C72, C66 to C73, L2 to L3, R48 to R44, R49 to R45, R50 to R46, R8 to R47, R6 to R48, R7 to R49, R9 to R50, U18 to U4, U16 to U5, U17 to U6, U3 to U7

Commit message: Add capacitor part library.
Parts:
- C64: value 2.2uF 6.3V -> 2.2uF 10V
- C67: value 100nF 16V -> 100nF 10V
- C72: value 22uF 16V -> 22uF 10V
Changed lines of the file:
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@@
 			)
 		)
-		(property "Value" "22uF 16V"
+		(property "Value" "22uF 10V"
 			(at 228.6 33.0262 0)
 			(effects
@@
 			)
 		)
-		(property "Value" "100nF 16V"
+		(property "Value" "100nF 10V"
 			(at 209.55 44.4562 0)
 			(effects
@@
 			)
 		)
-		(property "Value" "2.2uF 6.3V"
+		(property "Value" "2.2uF 10V"
 			(at 146.05 33.0262 0)
 			(effects

Commit message: Normalise capacitors
- Add capacitor parts to library.
- Replace all placeholder capacitors
  with the actual part numbers.
Parts:
- removed C59, C61, C62, C63, C65, C66, C68, C70, C71: 10uF 10V, symbol Device:C_Small
- removed C60: 100pF 30V, symbol Device:C_Small
- removed C64, C69, C73: 2.2uF 10V, symbol Device:C_Small
- removed C67: 100nF 10V, symbol Device:C_Small
- removed C72: 22uF 10V, symbol Device:C_Small
- added C59, C61, C62, C63, C65, C66, C68, C70, C71: 10uF 10V, Capacitor_SMD:C_0603_1608Metric, symbol symbol-library-capacitors:CC0603MRX5R6BB106
- added C60, C67: 100nF 10V, Capacitor_SMD:C_0402_1005Metric, symbol symbol-library-capacitors:CC0402KRX7R6BB104
- added C64, C69, C73: 2.2uF 10V, Capacitor_SMD:C_0402_1005Metric, symbol symbol-library-capacitors:CC0402KRX5R6BB225
- added C72: 22uF 10V, Capacitor_SMD:C_0603_1608Metric, symbol symbol-library-capacitors:CC0603MPX5R6BB226
Connections:
- net 1V8: now also C61.1, C62.1
- net 3V3: now also C65.1, C66.1
- net GND: now also C59.2, C60.2, C61.2, C62.2, C63.2, C64.2, C65.2, C66.2, C68.2, C69.2, C70.2, C71.2, C72.2, C73.2
- net VSYS: now also C59.1, C63.1
- net VSYS_IN: now also C68.1, C71.1
- net at U7.A5 (VDD): now also C64.1
- net at U7.C1 (BYP), U7.C2 (BYP): now also C72.1
- net at R50.1, U7.C5 (CSP), U7.D4 (BATT)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: now also C70.1, C73.1
- net at L3.1, U7.D1 (LX), U7.D2 (LX)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: now also C67.2
- net at U7.F1 (BST): now also C67.1
- net at U7.F2 (PVL): now also C69.1
- net at U4.7 (CT): now also C60.1

Commit message: Replace placeholder resistors
Parts:
- removed R44: 100R, symbol Device:R_Small_US
- removed R45, R46, R47: 10K, symbol Device:R_Small_US
- removed R48: 6.34K, symbol Device:R_Small_US
- removed R49: 4.42K, symbol Device:R_Small_US
- removed R50: 0.01R, symbol Device:R_Small_US
- added R40, R41, R45: 10K, Resistor_SMD:R_0402_1005Metric, symbol symbol-library-resistors:RC0402JR-0710KL
- added R42: 6.34K, Resistor_SMD:R_0402_1005Metric, symbol symbol-library-resistors:RC0402FR-076K34L
- added R43: 4.42K, Resistor_SMD:R_0402_1005Metric, symbol symbol-library-resistors:RC0402FR-074K42L
- added R44: 100R, Resistor_SMD:R_0402_1005Metric, symbol symbol-library-resistors:RC0402JR-07100RL
- added R46: 0.01R, Resistor_SMD:R_0402_1005Metric, symbol symbol-library-resistors:PE0402FRF7W0R01L
Connections:
- net 3V3: now also R40.1, R41.1
- net ALRT: now also R40.2
- net CHGEN: now also R41.2
- net GND: now also R42.1, R43.1
- net SYS_PGOOD: now also R45.2
- net VBAT: now also R46.2
- net VSYS: now also R44.1, R45.1
- net at U7.A1 (VCHG): now also R42.2
- net at U7.A2 (ICHG): now also R43.2
- net at C70.1, C73.1, U7.C5 (CSP)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: now also R46.1
- net at U4.5 (QOD): now also R44.2

Commit message: Add footprints
- Inductors
- Switches
- Buttons
Parts:
- removed J3: Conn_01x03, symbol Connector_Generic:Conn_01x03
- removed L3: 470nH (HTGH25201T-R47MSR-68), symbol Device:L
- removed SW1: SW_SPDT, symbol Switch:SW_SPDT
- added J3: S3B-PH-SM4-TB, footprint-library:S3B-PH-SM4-TB, symbol symbol-library:S3B-PH-SM4-TB
- added L4: 470nH 4.3A 0.025R, footprint-library:HMLQ25201T-R47MSR, symbol symbol-library-inductors:HMLQ25201T-R47MSR
- added SW1: 450404015514, footprint-library:450404015514, symbol symbol-library:450404015514
- renumbered R40 to R46, R41 to R47, R42 to R48, R43 to R49, R46 to R50
Connections:
- net GND: now also J3.2 (Pin_2), J3.MP (MountPin), SW1.3 (C)
- net VBAT: now also J3.3 (Pin_3)
- net VSYS_IN: now also L4.2, SW1.2 (B)
- net BAT_NTC: now reaches U7.A4 (THM)
- net BAT_NTC: now also J3.1 (Pin_1)
- net at C67.2, U7.D1 (LX), U7.D2 (LX)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: now also L4.1
- net at U4.8 (ON): now also SW1.1 (A)

Commit message: Fix footprint DRC errors.
Connections:
- net GND: now also SW1.4 (GND)
Changed lines of the file:
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@@
 	)
 	(junction
+		(at 36.83 137.16)
+		(diameter 0)
+		(color 0 0 0 0)
+	)
+	(junction
 		(at 219.71 67.31)
 		(diameter 0)
@@
 	)
 	(junction
-		(at 24.13 101.6)
+		(at 21.59 101.6)
 		(diameter 0)
 		(color 0 0 0 0)
@@
 	)
 	(junction
-		(at 24.13 99.06)
+		(at 21.59 99.06)
 		(diameter 0)
 		(color 0 0 0 0)
@@
 	(wire
 		(pts
-			(xy 35.56 129.54) (xy 36.83 129.54)
-		)
-		(stroke
-			(width 0)
-			(type default)
-		)
-	)
-	(wire
-		(pts
 			(xy 24.13 162.56) (xy 24.13 163.83)
 		)
@@
 	(wire
 		(pts
+			(xy 29.21 137.16) (xy 36.83 137.16)
+		)
+		(stroke
+			(width 0)
+			(type default)
+		)
+	)
+	(wire
+		(pts
 			(xy 67.31 124.46) (xy 67.31 125.73)
 		)
@@
 	(wire
 		(pts
-			(xy 25.4 127) (xy 24.13 127)
-		)
-		(stroke
-			(width 0)
-			(type default)
-		)
-	)
-	(wire
-		(pts
 			(xy 227.33 59.69) (xy 233.68 59.69)
 		)
@@
 	(wire
 		(pts
-			(xy 24.13 97.79) (xy 24.13 99.06)
+			(xy 21.59 97.79) (xy 21.59 99.06)
 		)
 		(stroke
@@
 	(wire
 		(pts
-			(xy 24.13 99.06) (xy 24.13 101.6)
+			(xy 21.59 99.06) (xy 21.59 101.6)
 		)
 		(stroke
@@
 	(wire
 		(pts
+			(xy 35.56 132.08) (xy 36.83 132.08)
+		)
+		(stroke
+			(width 0)
+			(type default)
+		)
+	)
+	(wire
+		(pts
 			(xy 207.01 48.26) (xy 217.17 48.26)
 		)
@@
 	(wire
 		(pts
-			(xy 24.13 99.06) (xy 38.1 99.06)
+			(xy 21.59 99.06) (xy 38.1 99.06)
 		)
 		(stroke
@@
 	(wire
 		(pts
+			(xy 36.83 137.16) (xy 36.83 139.7)
+		)
+		(stroke
+			(width 0)
+			(type default)
+		)
+	)
+	(wire
+		(pts
 			(xy 74.93 106.68) (xy 74.93 105.41)
 		)
@@
 		)
 	)
-	(bus
+	(wire
 		(pts
-			(xy 144.78 92.71) (xy 144.78 95.25)
+			(xy 21.59 128.27) (xy 22.86 128.27)
 		)
 		(stroke
@@
 	(bus
 		(pts
-			(xy 128.27 95.25) (xy 144.78 95.25)
+			(xy 144.78 92.71) (xy 144.78 95.25)
 		)
 		(stroke
@@
 		)
 	)
-	(wire
+	(bus
 		(pts
-			(xy 67.31 134.62) (xy 67.31 133.35)
+			(xy 128.27 95.25) (xy 144.78 95.25)
 		)
 		(stroke
@@
 	(wire
 		(pts
-			(xy 71.12 157.48) (xy 71.12 156.21)
+			(xy 67.31 134.62) (xy 67.31 133.35)
 		)
 		(stroke
@@
 	(wire
 		(pts
-			(xy 166.37 163.83) (xy 166.37 165.1)
+			(xy 71.12 157.48) (xy 71.12 156.21)
 		)
 		(stroke
@@
 	(wire
 		(pts
-			(xy 24.13 127) (xy 24.13 101.6)
+			(xy 166.37 163.83) (xy 166.37 165.1)
 		)
 		(stroke
@@
 	(wire
 		(pts
-			(xy 143.51 176.53) (xy 166.37 176.53)
+			(xy 21.59 101.6) (xy 21.59 128.27)
 		)
 		(stroke
@@
 	(wire
 		(pts
-			(xy 36.83 129.54) (xy 36.83 130.81)
+			(xy 143.51 176.53) (xy 166.37 176.53)
 		)
 		(stroke
@@
 	(wire
 		(pts
+			(xy 29.21 135.89) (xy 29.21 137.16)
+		)
+		(stroke
+			(width 0)
+			(type default)
+		)
+	)
+	(wire
+		(pts
 			(xy 273.05 74.93) (xy 273.05 72.39)
 		)
@@
 	(wire
 		(pts
+			(xy 36.83 132.08) (xy 36.83 137.16)
+		)
+		(stroke
+			(width 0)
+			(type default)
+		)
+	)
+	(wire
+		(pts
 			(xy 227.33 86.36) (xy 227.33 87.63)
 		)
@@
 	(wire
 		(pts
-			(xy 24.13 101.6) (xy 38.1 101.6)
+			(xy 21.59 101.6) (xy 38.1 101.6)
 		)
 		(stroke
@@
 	(symbol
 		(lib_id "symbol-library:450404015514")
-		(at 30.48 127 0)
+		(at 25.4 123.19 0)
 		(unit 1)
 		(exclude_from_sim no)
@@
 		(on_board yes)
 		(dnp no)
-		(fields_autoplaced yes)
 		(property "Reference" "SW1"
-			(at 30.48 118.11 0)
+			(at 27.178 120.396 0)
 			(effects
 				(font
@@
 		)
 		(property "Value" "450404015514"
-			(at 30.48 120.65 0)
+			(at 30.988 122.174 0)
 			(effects
 				(font
@@
 		)
 		(property "Footprint" "footprint-library:450404015514"
-			(at 30.48 127 0)
+			(at 25.4 123.19 0)
 			(effects
 				(font
@@
 		)
 		(property "Datasheet" "~"
-			(at 30.48 134.62 0)
+			(at 25.4 130.81 0)
 			(effects
 				(font
@@
 		)
 		(property "Description" "Switch, single pole double throw"
-			(at 30.48 127 0)
+			(at 25.4 123.19 0)
 			(effects
 				(font
@@
 		(pin "1"
 		)
+		(pin "4"
+		)
 		(instances
-			(project ""
+			(project "main-board"
 				(path "/c621b5fd-2ef7-4a67-960d-0ffc72b1245a/8c4d5296-af08-4575-a315-f8c9eefb13c6"
 					(reference "SW1")
@@
 	(symbol
 		(lib_id "power:VCC")
-		(at 24.13 97.79 0)
+		(at 21.59 97.79 0)
 		(unit 1)
 		(exclude_from_sim no)
@@
 		(fields_autoplaced yes)
 		(property "Reference" "#PWR088"
-			(at 24.13 101.6 0)
+			(at 21.59 101.6 0)
 			(effects
 				(font
@@
 		)
 		(property "Value" "VSYS_IN"
-			(at 24.13 92.71 0)
+			(at 21.59 92.71 0)
 			(effects
 				(font
@@
 		)
 		(property "Footprint" ""
-			(at 24.13 97.79 0)
+			(at 21.59 97.79 0)
 			(effects
 				(font
@@
 		)
 		(property "Datasheet" ""
-			(at 24.13 97.79 0)
+			(at 21.59 97.79 0)
 			(effects
 				(font
@@
 		)
 		(property "Description" "Power symbol creates a global label with name \"VCC\""
-			(at 24.13 97.79 0)
+			(at 21.59 97.79 0)
 			(effects
 				(font
@@
 	(symbol
 		(lib_id "power:GND")
-		(at 36.83 130.81 0)
+		(at 36.83 139.7 0)
 		(unit 1)
 		(exclude_from_sim no)
@@
 		(fields_autoplaced yes)
 		(property "Reference" "#PWR091"
-			(at 36.83 137.16 0)
+			(at 36.83 146.05 0)
 			(effects
 				(font
@@
 		)
 		(property "Value" "GND"
-			(at 36.83 135.89 0)
+			(at 36.83 144.78 0)
 			(effects
 				(font
@@
 		)
 		(property "Footprint" ""
-			(at 36.83 130.81 0)
+			(at 36.83 139.7 0)
 			(effects
 				(font
@@
 		)
 		(property "Datasheet" ""
-			(at 36.83 130.81 0)
+			(at 36.83 139.7 0)
 			(effects
 				(font
@@
 		)
 		(property "Description" "Power symbol creates a global label with name \"GND\" , ground"
-			(at 36.83 130.81 0)
+			(at 36.83 139.7 0)
 			(effects
 				(font
@@
 	)
 	(symbol
-		(lib_name "TPSM863253RDXR_1")
 		(lib_id "symbol-library:TPSM863253RDXR")
 		(at 123.19 154.94 0)
@@
 	)
 	(symbol
-		(lib_name "MPM3805GQB-18-Z_1")
 		(lib_id "symbol-library:MPM3805GQB-18-Z")
 		(at 45.72 153.67 0)

Commit message: Rough PCB component grouping and layout
Parts:
- added C108: 2.2uF 10V, Capacitor_SMD:C_0402_1005Metric, symbol symbol-library-capacitors:CC0402KRX5R6BB225
Connections:
- net GND: now also C108.2
- net VBUS: now also C108.1
Other:
- moved on the sheet: C64
Changed lines of the file:
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@@
 	)
 	(junction
+		(at 139.7 39.37)
+		(diameter 0)
+		(color 0 0 0 0)
+	)
+	(junction
 		(at 201.93 118.11)
 		(diameter 0)
@@
 	(wire
 		(pts
+			(xy 139.7 38.1) (xy 139.7 39.37)
+		)
+		(stroke
+			(width 0)
+			(type default)
+		)
+	)
+	(wire
+		(pts
 			(xy 96.52 76.2) (xy 163.83 76.2)
 		)
@@
 	(wire
 		(pts
+			(xy 139.7 45.72) (xy 139.7 46.99)
+		)
+		(stroke
+			(width 0)
+			(type default)
+		)
+	)
+	(wire
+		(pts
 			(xy 209.55 115.57) (xy 209.55 120.65)
 		)
@@
 	(wire
 		(pts
-			(xy 162.56 39.37) (xy 158.75 39.37)
+			(xy 162.56 39.37) (xy 139.7 39.37)
 		)
 		(stroke
@@
 	(wire
 		(pts
+			(xy 139.7 39.37) (xy 139.7 40.64)
+		)
+		(stroke
+			(width 0)
+			(type default)
+		)
+	)
+	(wire
+		(pts
 			(xy 96.52 78.74) (xy 113.03 78.74)
 		)
@@
 	(wire
 		(pts
-			(xy 143.51 29.21) (xy 143.51 27.94)
+			(xy 124.46 29.21) (xy 124.46 27.94)
 		)
 		(stroke
@@
 	(wire
 		(pts
-			(xy 143.51 27.94) (xy 163.83 27.94)
+			(xy 124.46 27.94) (xy 163.83 27.94)
 		)
 		(stroke
@@
 	(wire
 		(pts
-			(xy 143.51 35.56) (xy 143.51 34.29)
+			(xy 124.46 35.56) (xy 124.46 34.29)
 		)
 		(stroke
@@
 	)
 	(symbol
+		(lib_id "symbol-library-capacitors:CC0402KRX5R6BB225")
+		(at 139.7 43.18 0)
+		(unit 1)
+		(exclude_from_sim no)
+		(in_bom yes)
+		(on_board yes)
+		(dnp no)
+		(fields_autoplaced yes)
+		(property "Reference" "C108"
+			(at 142.24 41.9162 0)
+			(effects
+				(font
+					(size 1.27 1.27)
+				)
+				(justify left)
+			)
+		)
+		(property "Value" "2.2uF 10V"
+			(at 142.24 44.4562 0)
+			(effects
+				(font
+					(size 1.27 1.27)
+				)
+				(justify left)
+			)
+		)
+		(property "Footprint" "Capacitor_SMD:C_0402_1005Metric"
+			(at 139.7 43.18 0)
+			(effects
+				(font
+					(size 1.27 1.27)
+				)
+				(hide yes)
+			)
+		)
+		(property "Datasheet" "~"
+			(at 139.7 43.18 0)
+			(effects
+				(font
+					(size 1.27 1.27)
+				)
+				(hide yes)
+			)
+		)
+		(property "Description" "Unpolarized capacitor, small symbol"
+			(at 139.7 43.18 0)
+			(effects
+				(font
+					(size 1.27 1.27)
+				)
+				(hide yes)
+			)
+		)
+		(pin "2"
+		)
+		(pin "1"
+		)
+		(instances
+			(project "main-board"
+				(path "/c621b5fd-2ef7-4a67-960d-0ffc72b1245a/8c4d5296-af08-4575-a315-f8c9eefb13c6"
+					(reference "C108")
+					(unit 1)
+				)
+			)
+		)
+	)
+	(symbol
 		(lib_id "power:GND")
-		(at 143.51 35.56 0)
+		(at 124.46 35.56 0)
 		(unit 1)
 		(exclude_from_sim no)
@@
 		(fields_autoplaced yes)
 		(property "Reference" "#PWR0100"
-			(at 143.51 41.91 0)
+			(at 124.46 41.91 0)
 			(effects
 				(font
@@
 		)
 		(property "Value" "GND"
-			(at 143.51 40.64 0)
+			(at 124.46 40.64 0)
 			(effects
 				(font
@@
 		)
 		(property "Footprint" ""
-			(at 143.51 35.56 0)
+			(at 124.46 35.56 0)
 			(effects
 				(font
@@
 		)
 		(property "Datasheet" ""
-			(at 143.51 35.56 0)
+			(at 124.46 35.56 0)
 			(effects
 				(font
@@
 		)
 		(property "Description" "Power symbol creates a global label with name \"GND\" , ground"
-			(at 143.51 35.56 0)
+			(at 124.46 35.56 0)
 			(effects
 				(font
@@
 	)
 	(symbol
+		(lib_id "power:GND")
+		(at 139.7 46.99 0)
+		(unit 1)
+		(exclude_from_sim no)
+		(in_bom yes)
+		(on_board yes)
+		(dnp no)
+		(fields_autoplaced yes)
+		(property "Reference" "#PWR0160"
+			(at 139.7 53.34 0)
+			(effects
+				(font
+					(size 1.27 1.27)
+				)
+				(hide yes)
+			)
+		)
+		(property "Value" "GND"
+			(at 139.7 52.07 0)
+			(effects
+				(font
+					(size 1.27 1.27)
+				)
+			)
+		)
+		(property "Footprint" ""
+			(at 139.7 46.99 0)
+			(effects
+				(font
+					(size 1.27 1.27)
+				)
+				(hide yes)
+			)
+		)
+		(property "Datasheet" ""
+			(at 139.7 46.99 0)
+			(effects
+				(font
+					(size 1.27 1.27)
+				)
+				(hide yes)
+			)
+		)
+		(property "Description" "Power symbol creates a global label with name \"GND\" , ground"
+			(at 139.7 46.99 0)
+			(effects
+				(font
+					(size 1.27 1.27)
+				)
+				(hide yes)
+			)
+		)
+		(pin "1"
+		)
+		(instances
+			(project "main-board"
+				(path "/c621b5fd-2ef7-4a67-960d-0ffc72b1245a/8c4d5296-af08-4575-a315-f8c9eefb13c6"
+					(reference "#PWR0160")
+					(unit 1)
+				)
+			)
+		)
+	)
+	(symbol
 		(lib_id "power:VCC")
 		(at 21.59 97.79 0)
@@
 	(symbol
 		(lib_id "power:VCC")
-		(at 158.75 39.37 0)
+		(at 139.7 38.1 0)
 		(unit 1)
 		(exclude_from_sim no)
@@
 		(fields_autoplaced yes)
 		(property "Reference" "#PWR0101"
-			(at 158.75 43.18 0)
+			(at 139.7 41.91 0)
 			(effects
 				(font
@@
 		)
 		(property "Value" "VBUS"
-			(at 158.75 34.29 0)
+			(at 139.7 33.02 0)
 			(effects
 				(font
@@
 		)
 		(property "Footprint" ""
-			(at 158.75 39.37 0)
+			(at 139.7 38.1 0)
 			(effects
 				(font
@@
 		)
 		(property "Datasheet" ""
-			(at 158.75 39.37 0)
+			(at 139.7 38.1 0)
 			(effects
 				(font
@@
 		)
 		(property "Description" "Power symbol creates a global label with name \"VCC\""
-			(at 158.75 39.37 0)
+			(at 139.7 38.1 0)
 			(effects
 				(font
@@
 	(symbol
 		(lib_id "symbol-library-capacitors:CC0402KRX5R6BB225")
-		(at 143.51 31.75 0)
+		(at 124.46 31.75 0)
 		(unit 1)
 		(exclude_from_sim no)
@@
 		(fields_autoplaced yes)
 		(property "Reference" "C64"
-			(at 146.05 30.4862 0)
+			(at 127 30.4862 0)
 			(effects
 				(font
@@
 		)
 		(property "Value" "2.2uF 10V"
-			(at 146.05 33.0262 0)
+			(at 127 33.0262 0)
 			(effects
 				(font
@@
 		)
 		(property "Footprint" "Capacitor_SMD:C_0402_1005Metric"
-			(at 143.51 31.75 0)
+			(at 124.46 31.75 0)
 			(effects
 				(font
@@
 		)
 		(property "Datasheet" "~"
-			(at 143.51 31.75 0)
+			(at 124.46 31.75 0)
 			(effects
 				(font
@@
 		)
 		(property "Description" "Unpolarized capacitor, small symbol"
-			(at 143.51 31.75 0)
+			(at 124.46 31.75 0)
 			(effects
 				(font
