File: projects/main-board/mcu.kicad_sch (KiCad schematic)
At the start: 107 parts, among them J1 TC2030, J2 TC2030, U1 STM32N657X0HxQ

Commit message: Update render.
Connections:
- net BUTTONS.B12: no longer names the net of U1.T1 (PF12)
- net BUTTONS.B13: no longer names the net of U1.R2 (PF13)
- net BUTTONS.B14: no longer names the net of U1.N2 (PF14)
- net BUTTONS.B15: no longer names the net of U1.N1 (PF15)
Changed lines of the file:
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@@
 	(wire
 		(pts
-			(xy 435.61 85.09) (xy 457.2 85.09)
-		)
-		(stroke
-			(width 0)
-			(type default)
-		)
-	)
-	(wire
-		(pts
 			(xy 97.79 266.7) (xy 97.79 267.97)
 		)
@@
 		)
 	)
-	(wire
-		(pts
-			(xy 435.61 77.47) (xy 457.2 77.47)
-		)
-		(stroke
-			(width 0)
-			(type default)
-		)
-	)
 	(bus
 		(pts
@@
 	(wire
 		(pts
-			(xy 435.61 80.01) (xy 457.2 80.01)
-		)
-		(stroke
-			(width 0)
-			(type default)
-		)
-	)
-	(wire
-		(pts
 			(xy 107.95 194.31) (xy 107.95 195.58)
 		)
@@
 	(wire
 		(pts
-			(xy 435.61 82.55) (xy 457.2 82.55)
-		)
-		(stroke
-			(width 0)
-			(type default)
-		)
-	)
-	(wire
-		(pts
 			(xy 135.89 354.33) (xy 135.89 355.6)
 		)
@@
 		)
 	)
-	(label "BUTTONS.B14"
-		(at 444.5 82.55 0)
-		(effects
-			(font
-				(size 1.27 1.27)
-			)
-			(justify left bottom)
-		)
-	)
 	(label "I2C4.SDA"
 		(at 265.43 300.99 0)
@@
 		)
 	)
-	(label "BUTTONS{B[0..15]}"
+	(label "BUTTONS{B[0..11]}"
 		(at 205.74 100.33 0)
 		(effects
@@
 		)
 	)
-	(label "BUTTONS.B15"
-		(at 444.5 85.09 0)
-		(effects
-			(font
-				(size 1.27 1.27)
-			)
-			(justify left bottom)
-		)
-	)
 	(label "RAM_HEXASPI.DQS1"
 		(at 454.66 250.19 0)
@@
 		)
 	)
-	(label "BUTTONS.B13"
-		(at 444.5 80.01 0)
-		(effects
-			(font
-				(size 1.27 1.27)
-			)
-			(justify left bottom)
-		)
-	)
 	(label "PMIC_INPUT_VALID"
 		(at 308.61 215.9 0)
@@
 		(effects
 			(font
-				(size 1.27 1.27)
-			)
-			(justify left bottom)
-		)
-	)
-	(label "BUTTONS.B12"
-		(at 444.5 77.47 0)
-		(effects
-			(font
