File: projects/main-board/mcu.kicad_sch (KiCad schematic)
At the start: 107 parts, among them J1 TC2030, J2 TC2030, U1 STM32N657X0HxQ

Commit message: Update render
Connections:
- net BUTTONS.B10: no longer names the net of U1.L4 (PF10)
- net BUTTONS.B11: no longer names the net of U1.P3 (PF11)
Changed lines of the file:
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@@
 	(wire
 		(pts
-			(xy 435.61 72.39) (xy 457.2 72.39)
-		)
-		(stroke
-			(width 0)
-			(type default)
-		)
-	)
-	(wire
-		(pts
 			(xy 63.5 344.17) (xy 63.5 346.71)
 		)
@@
 	(wire
 		(pts
-			(xy 435.61 74.93) (xy 457.2 74.93)
-		)
-		(stroke
-			(width 0)
-			(type default)
-		)
-	)
-	(wire
-		(pts
 			(xy 63.5 251.46) (xy 62.23 251.46)
 		)
@@
 		)
 	)
-	(label "BUTTONS{B[0..11]}"
+	(label "BUTTONS{B[0..9]}"
 		(at 205.74 100.33 0)
 		(effects
@@
 		)
 	)
-	(label "BUTTONS.B10"
-		(at 444.5 72.39 0)
-		(effects
-			(font
-				(size 1.27 1.27)
-			)
-			(justify left bottom)
-		)
-	)
 	(label "MOTOR_PWR_EN"
 		(at 205.74 80.01 0)
@@
 		(effects
 			(font
-				(size 1.27 1.27)
-			)
-			(justify left bottom)
-		)
-	)
-	(label "BUTTONS.B11"
-		(at 444.5 74.93 0)
-		(effects
-			(font

Commit message: Main board PCB layout and routing
- Add 48MHz crystal for STM32
- Add 32kHz crystal for STM32
- Started laying out and routing board
Parts:
- added C109, C110: 9pF 50V, Capacitor_SMD:C_0402_1005Metric, symbol symbol-library-capacitors:CC0402CRNPO9BN9R0
- added C115, C116: 8pF 50V, Capacitor_SMD:C_0402_1005Metric, symbol symbol-library-capacitors:CC0402CRNPO9BN8R0
- added R61, R62, R64, R65: 0R, Resistor_SMD:R_0402_1005Metric, symbol symbol-library-resistors:RC0402FR-070RL
- added Y2: ABM11W-48.0000MHZ-8-K1Z-T3, footprint-library:ABM11W300000MHZ4B1UT3, symbol symbol-library:ABM11W-48.0000MHZ-8-K1Z-T3
- added Y3: ABS06-32.768KHZ-9-1-T, footprint-library:ABS06, symbol symbol-library:ABS06-32.768KHZ-9-1-T
Connections:
- net GND: now also C109.2, C110.2, C115.2, C116.2, Y2.2 (GND), Y2.4 (GND)
- net at U1.A7 (PH0-OSC_IN(PH0)): now also R61.1
- net at U1.B7 (PH1-OSC_OUT(PH1)): now also R62.1
- net at U1.C1 (PC15-OSC32_OUT(OSC32_OUT)): now also R64.2
- net at U1.D1 (PC14-OSC32_IN(OSC32_IN)): now also R65.2
- net USB.DM renamed USB.DN
- new net: C109.1, R65.1, Y3.1
- new net: C116.1, R62.2, Y2.3
- new net: C115.1, R61.2, Y2.1
- new net: C110.1, R64.1, Y3.2

Commit message: Routed LCD signals
Connections:
- net BUTTONS.B1: now also U1.T1 (PF12); no longer U1.P4 (PF1)
- net BUTTONS.B2: now also U1.P2 (PG4); no longer U1.N4 (PF2)
- net BUTTONS.B3: now also U1.F4 (PH4); no longer U1.M2 (PF3)
- net BUTTONS.B6: now also U1.L1 (PG7); no longer U1.L5 (PF6)
- net DEBUG_UART.RX: now also U1.C14 (PD14); no longer U1.R7 (PA10)
- net DEBUG_UART.TX: now also U1.D15 (PB9); no longer U1.P7 (PA9)
- net ESP32_GPIO.3: now also U1.A13 (PD10); no longer U1.A9 (PC1)
- net ESP32_GPIO.9: now also U1.A14 (PD1); no longer U1.A8 (PC10)
- net LCD.B2: now also U1.U7 (PA12); no longer U1.C16 (PB2)
- net LCD.B3: now also U1.T7 (PA11); no longer U1.L3 (PG6)
- net LCD.B4: now also U1.R7 (PA10); no longer U1.B1 (PH3)
- net LCD.B5: now also U1.P7 (PA9); no longer U1.B2 (PH6)
- net LCD.CLK: now also U1.R8 (PA5); no longer U1.C15 (PB13)
- net LCD.EN: now also U1.U14 (PA4); no longer U1.D3 (PQ3)
- net LCD.G4: now also U1.T10 (PG10); no longer U1.D17 (PB15)
- net LCD.HSYNC: now also U1.P8 (PA6); no longer U1.B17 (PB14)
- net LCD.R1: now also U1.L4 (PF10); no longer U1.H14 (PD9)
- net LCD.R2: now also U1.U12 (PB5(JTDO/TRACESWO)); no longer U1.B14 (PD15)
- net LCD.R4: now also U1.M2 (PF3); no longer U1.F4 (PH4)
- net LCD.R7: now also U1.T13 (PG9); no longer U1.E14 (PD8)
- net LEFT_MOTOR_PWM: now also U1.D5 (PQ5); no longer U1.R8 (PA5)
- net PMIC_ALERT: now also U1.R2 (PF13); no longer U1.D13 (PD0)
- net PMIC_CHARGE_EN: now also U1.R1 (PG3); no longer U1.E13 (PD3)
- net PMIC_INPUT_VALID: now also U1.N1 (PF15); no longer U1.C12 (PD2)
- net PMIC_STATUS: now also U1.N2 (PF14); no longer U1.A14 (PD1)
- net RIGHT_MOTOR_PWM: now also U1.G5 (PQ7); no longer U1.P8 (PA6)
- net VBAT: no longer C12.1
- net at R3.2, R4.1, U1.E1 (VBAT): now also C12.1
- no-connect marks 17 -> 68
Other:
- note added: "TIM8_CH2"
- note added: "TIM8_CH3"
- note added: "USART10_RX"
- note added: "USART10_TX"
- note removed: "TIM10_CH1"
- note removed: "TIM13_CH1"
- note removed: "USART1_RX"
- note removed: "USART1_TX"
- moved on the sheet: C115, C116, C12, R3, R4, R61, R62, Y2

Commit message: More routing of main board
Parts:
- removed NT2, NT6: NetTie_2, symbol Device:NetTie_2
Connections:
- net 1V8: now also L2.1, L3.1
- net BUTTONS.B5: now also U1.B1 (PH3); no longer U1.M3 (PF5)
- net BUTTONS.B8: now also U1.B2 (PH6); no longer U1.N3 (PF8)
- net ESP32_EN: now also U1.B17 (PB14); no longer U1.F13 (PB3)
- net MOTOR_PWR_EN: now also U1.A16 (PE9)
- net VDDA18PMU: now also C13.1, L2.2; no longer L2.1
- net VDDSMPS: now also C16.1, C24.1, C32.1, C39.1, C44.1, C47.1, L3.2; no longer L3.1
- no-connect marks 68 -> 72
Other:
- moved on the sheet: C16, C24, C32, C39, C44, C47, L3
