File: projects/main-board/ram.kicad_sch (KiCad schematic)
At the start: 6 parts

Commit message: Updated schematics with new symbols
Parts:
- removed U2: ~, symbol symbol-library:APS256XXN-OBR-BG
- added U1: APS256XXN-OBR-BG, footprint-library:APS256XXN-OBR-BG, symbol symbol-library:APS256XXN-OBR-BG
Connections:
- net 1V8: now also U1.D1 (VDD), U1.E4 (VDD)
- net GND: now also U1.C1 (VSS), U1.E5 (VSS)
- net RAM_HEXASPI.CLK: now also U1.B2 (CLK)
- net RAM_HEXASPI.CS_N: now also U1.A3 (CE#)
- net RAM_HEXASPI.D0: now also U1.D3 (ADQ0)
- net RAM_HEXASPI.D1: now also U1.D2 (ADQ1)
- net RAM_HEXASPI.D10: now also U1.A2 (DQ10)
- net RAM_HEXASPI.D11: now also U1.A4 (DQ11)
- net RAM_HEXASPI.D12: now also U1.A5 (DQ12)
- net RAM_HEXASPI.D13: now also U1.B4 (DQ13)
- net RAM_HEXASPI.D14: now also U1.B5 (DQ14)
- net RAM_HEXASPI.D15: now also U1.C5 (DQ15)
- net RAM_HEXASPI.D2: now also U1.C4 (ADQ2)
- net RAM_HEXASPI.D3: now also U1.D4 (ADQ3)
- net RAM_HEXASPI.D4: now also U1.D5 (ADQ4)
- net RAM_HEXASPI.D5: now also U1.E3 (ADQ5)
- net RAM_HEXASPI.D6: now also U1.E2 (ADQ6)
- net RAM_HEXASPI.D7: now also U1.E1 (ADQ7)
- net RAM_HEXASPI.D8: now also U1.C2 (DQ8)
- net RAM_HEXASPI.D9: now also U1.B1 (DQ9)
- net RAM_HEXASPI.DQS0: now also U1.C3 (DQS/DM0)
- net RAM_HEXASPI.DQS1: now also U1.B3 (DQS/DM1)
Changed lines of the file:
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@@
-	)
-	(junction
-		(at 158.75 64.77)
-		(diameter 0)
-		(color 0 0 0 0)
 	)
 	(junction
@@
 	(junction
 		(at 73.66 64.77)
+		(diameter 0)
+		(color 0 0 0 0)
+	)
+	(junction
+		(at 158.75 64.77)
 		(diameter 0)
 		(color 0 0 0 0)
@@
 	)
 	(symbol
+		(lib_name "APS256XXN-OBR-BG_1")
+		(lib_id "symbol-library:APS256XXN-OBR-BG")
+		(at 161.29 69.85 0)
+		(unit 1)
+		(exclude_from_sim no)
+		(in_bom yes)
+		(on_board yes)
+		(dnp no)
+		(property "Reference" "U1"
+			(at 162.306 61.214 0)
+			(effects
+				(font
+					(size 1.27 1.27)
+				)
+			)
+		)
+		(property "Value" "APS256XXN-OBR-BG"
+			(at 170.18 139.954 0)
+			(effects
+				(font
+					(size 1.27 1.27)
+				)
+			)
+		)
+		(property "Footprint" "footprint-library:APS256XXN-OBR-BG"
+			(at 176.53 141.478 0)
+			(effects
+				(font
+					(size 1.27 1.27)
+				)
+				(hide yes)
+			)
+		)
+		(property "Datasheet" ""
+			(at 161.29 69.85 0)
+			(effects
+				(font
+					(size 1.27 1.27)
+				)
+				(hide yes)
+			)
+		)
+		(property "Description" ""
+			(at 161.29 69.85 0)
+			(effects
+				(font
+					(size 1.27 1.27)
+				)
+				(hide yes)
+			)
+		)
+		(pin "D1"
+		)
+		(pin "E4"
+		)
+		(pin "A3"
+		)
+		(pin "B2"
+		)
+		(pin "C3"
+		)
+		(pin "B3"
+		)
+		(pin "D3"
+		)
+		(pin "D2"
+		)
+		(pin "C4"
+		)
+		(pin "D4"
+		)
+		(pin "D5"
+		)
+		(pin "E3"
+		)
+		(pin "E2"
+		)
+		(pin "E1"
+		)
+		(pin "C2"
+		)
+		(pin "B1"
+		)
+		(pin "A2"
+		)
+		(pin "A4"
+		)
+		(pin "A5"
+		)
+		(pin "B4"
+		)
+		(pin "B5"
+		)
+		(pin "C5"
+		)
+		(pin "C1"
+		)
+		(pin "E5"
+		)
+		(instances
+			(project ""
+				(path "/c621b5fd-2ef7-4a67-960d-0ffc72b1245a/a4a3f1ff-d673-4de4-9dae-3d1051c84f77"
+					(reference "U1")
+					(unit 1)
+				)
+			)
+		)
+	)
+	(symbol
 		(lib_id "Device:C_Small")
 		(at 87.63 68.58 0)
@@
 					(unit 1)
 				)
-			)
-		)
-	)
-	(symbol
-		(lib_id "symbol-library:APS256XXN-OBR-BG")
-		(at 161.29 69.85 0)
-		(unit 1)
-		(exclude_from_sim no)
-		(in_bom yes)
-		(on_board yes)
-		(dnp no)
-		(property "Reference" "U2"
-			(at 162.306 60.96 0)
-			(effects
-				(font
-					(size 1.27 1.27)
-				)
-			)
-		)
-		(property "Value" "~"
-			(at 168.402 60.706 0)
-			(effects
-				(font
-					(size 1.27 1.27)
-				)
-			)
-		)
-		(property "Footprint" ""
-			(at 161.29 69.85 0)
-			(effects
-				(font
-					(size 1.27 1.27)
-				)
-				(hide yes)
-			)
-		)
-		(property "Datasheet" ""
-			(at 161.29 69.85 0)
-			(effects
-				(font
-					(size 1.27 1.27)
-				)
-				(hide yes)
-			)
-		)
-		(property "Description" ""
-			(at 161.29 69.85 0)
-			(effects
-				(font
-					(size 1.27 1.27)
-				)
-				(hide yes)
-			)
-		)
-		(pin "D1"
-		)
-		(pin "E4"
-		)
-		(pin "A3"
-		)
-		(pin "B2"
-		)
-		(pin "C3"
-		)
-		(pin "D3"
-		)
-		(pin "D2"
-		)
-		(pin "C4"
-		)
-		(pin "D4"
-		)
-		(pin "D5"
-		)
-		(pin "E3"
-		)
-		(pin "E2"
-		)
-		(pin "E1"
-		)
-		(pin "C2"
-		)
-		(pin "B1"
-		)
-		(pin "A2"
-		)
-		(pin "A4"
-		)
-		(pin "A5"
-		)
-		(pin "B4"
-		)
-		(pin "B5"
-		)
-		(pin "C5"
-		)
-		(pin "C1"
-		)
-		(pin "E5"
-		)
-		(pin "B3"
-		)
-		(instances
-			(project ""
-				(path "/c621b5fd-2ef7-4a67-960d-0ffc72b1245a/a4a3f1ff-d673-4de4-9dae-3d1051c84f77"
-					(reference "U2")
-					(unit 1)
-				)

Commit message: Re-annotate schematics.
Parts:
- renumbered R1 to R40, U1 to U2
Changed lines of the file:
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@@
 		(dnp no)
 		(fields_autoplaced yes)
-		(property "Reference" "R1"
+		(property "Reference" "R40"
 			(at 140.97 69.8499 0)
 			(effects
@@
 			(project ""
 				(path "/c621b5fd-2ef7-4a67-960d-0ffc72b1245a/a4a3f1ff-d673-4de4-9dae-3d1051c84f77"
-					(reference "R1")
+					(reference "R40")
 					(unit 1)
 				)
@@
 		(dnp no)
 		(fields_autoplaced yes)
-		(property "Reference" "#PWR075"
+		(property "Reference" "#PWR082"
 			(at 73.66 68.58 0)
 			(effects
@@
 			(project "main-board"
 				(path "/c621b5fd-2ef7-4a67-960d-0ffc72b1245a/a4a3f1ff-d673-4de4-9dae-3d1051c84f77"
-					(reference "#PWR075")
+					(reference "#PWR082")
 					(unit 1)
 				)
@@
 		(on_board yes)
 		(dnp no)
-		(property "Reference" "U1"
+		(property "Reference" "U2"
 			(at 162.306 61.214 0)
 			(effects
@@
 			(project ""
 				(path "/c621b5fd-2ef7-4a67-960d-0ffc72b1245a/a4a3f1ff-d673-4de4-9dae-3d1051c84f77"
-					(reference "U1")
+					(reference "U2")
 					(unit 1)
 				)
@@
 		(dnp no)
 		(fields_autoplaced yes)
-		(property "Reference" "#PWR076"
+		(property "Reference" "#PWR083"
 			(at 73.66 78.74 0)
 			(effects
@@
 			(project "main-board"
 				(path "/c621b5fd-2ef7-4a67-960d-0ffc72b1245a/a4a3f1ff-d673-4de4-9dae-3d1051c84f77"
-					(reference "#PWR076")
+					(reference "#PWR083")
 					(unit 1)
 				)
@@
 		(dnp no)
 		(fields_autoplaced yes)
-		(property "Reference" "#PWR074"
+		(property "Reference" "#PWR084"
 			(at 189.23 143.51 0)
 			(effects
@@
 			(project ""
 				(path "/c621b5fd-2ef7-4a67-960d-0ffc72b1245a/a4a3f1ff-d673-4de4-9dae-3d1051c84f77"
-					(reference "#PWR074")
-					(unit 1)
-				)
+					(reference "#PWR084")
+					(unit 1)
+				)

Commit message: Add capacitor part library.
Parts:
- C51, C52: value 4.7uF 6.3V -> 4.7uF 10V
Changed lines of the file:
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@@
 			)
 		)
-		(property "Value" "4.7uF 6.3V"
+		(property "Value" "4.7uF 10V"
 			(at 104.14 69.8562 0)
 			(effects
@@
 			)
 		)
-		(property "Value" "4.7uF 6.3V"
+		(property "Value" "4.7uF 10V"
 			(at 118.11 69.8562 0)
 			(effects

Commit message: Normalise capacitors
- Add capacitor parts to library.
- Replace all placeholder capacitors
  with the actual part numbers.
Parts:
- removed C49, C50: 100nF 10V, symbol Device:C_Small
- removed C51, C52: 4.7uF 10V, symbol Device:C_Small
- added C49, C50: 100nF 10V, Capacitor_SMD:C_0402_1005Metric, symbol symbol-library-capacitors:CC0402KRX7R6BB104
- added C51, C52: 4.7uF 10V, Capacitor_SMD:C_0402_1005Metric, symbol symbol-library-capacitors:CC0402MRX5R6BB475
Connections:
- net 1V8: now also C49.1, C50.1, C51.1, C52.1
- net GND: now also C49.2, C50.2, C51.2, C52.2
Changed lines of the file:
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@@
 	)
 	(symbol
-		(lib_id "Device:C_Small")
-		(at 101.6 68.58 0)
-		(unit 1)
-		(exclude_from_sim no)
-		(in_bom yes)
-		(on_board yes)
-		(dnp no)
-		(fields_autoplaced yes)
-		(property "Reference" "C51"
-			(at 104.14 67.3162 0)
+		(lib_id "symbol-library-capacitors:CC0402MRX5R6BB475")
+		(at 115.57 68.58 0)
+		(unit 1)
+		(exclude_from_sim no)
+		(in_bom yes)
+		(on_board yes)
+		(dnp no)
+		(fields_autoplaced yes)
+		(property "Reference" "C52"
+			(at 118.11 67.3162 0)
 			(effects
 				(font
@@
 		)
 		(property "Value" "4.7uF 10V"
-			(at 104.14 69.8562 0)
-			(effects
-				(font
-					(size 1.27 1.27)
-				)
-				(justify left)
-			)
-		)
-		(property "Footprint" ""
-			(at 101.6 68.58 0)
+			(at 118.11 69.8562 0)
+			(effects
+				(font
+					(size 1.27 1.27)
+				)
+				(justify left)
+			)
+		)
+		(property "Footprint" "Capacitor_SMD:C_0402_1005Metric"
+			(at 115.57 68.58 0)
 			(effects
 				(font
@@
 		)
 		(property "Datasheet" "~"
-			(at 101.6 68.58 0)
+			(at 115.57 68.58 0)
 			(effects
 				(font
@@
 		)
 		(property "Description" "Unpolarized capacitor, small symbol"
-			(at 101.6 68.58 0)
-			(effects
-				(font
-					(size 1.27 1.27)
-				)
-				(hide yes)
-			)
+			(at 115.57 68.58 0)
+			(effects
+				(font
+					(size 1.27 1.27)
+				)
+				(hide yes)
+			)
+		)
+		(pin "1"
 		)
 		(pin "2"
 		)
-		(pin "1"
-		)
 		(instances
 			(project "main-board"
 				(path "/c621b5fd-2ef7-4a67-960d-0ffc72b1245a/a4a3f1ff-d673-4de4-9dae-3d1051c84f77"
-					(reference "C51")
+					(reference "C52")
 					(unit 1)
 				)
@@
 		(dnp no)
 		(fields_autoplaced yes)
-		(property "Reference" "#PWR082"
+		(property "Reference" "#PWR081"
 			(at 73.66 68.58 0)
 			(effects
@@
 			(project "main-board"
 				(path "/c621b5fd-2ef7-4a67-960d-0ffc72b1245a/a4a3f1ff-d673-4de4-9dae-3d1051c84f77"
-					(reference "#PWR082")
+					(reference "#PWR081")
 					(unit 1)
 				)
@@
 	)
 	(symbol
-		(lib_id "Device:C_Small")
+		(lib_id "symbol-library-capacitors:CC0402KRX7R6BB104")
+		(at 73.66 68.58 0)
+		(unit 1)
+		(exclude_from_sim no)
+		(in_bom yes)
+		(on_board yes)
+		(dnp no)
+		(fields_autoplaced yes)
+		(property "Reference" "C49"
+			(at 76.2 67.3162 0)
+			(effects
+				(font
+					(size 1.27 1.27)
+				)
+				(justify left)
+			)
+		)
+		(property "Value" "100nF 10V"
+			(at 76.2 69.8562 0)
+			(effects
+				(font
+					(size 1.27 1.27)
+				)
+				(justify left)
+			)
+		)
+		(property "Footprint" "Capacitor_SMD:C_0402_1005Metric"
+			(at 73.66 68.58 0)
+			(effects
+				(font
+					(size 1.27 1.27)
+				)
+				(hide yes)
+			)
+		)
+		(property "Datasheet" "~"
+			(at 73.66 68.58 0)
+			(effects
+				(font
+					(size 1.27 1.27)
+				)
+				(hide yes)
+			)
+		)
+		(property "Description" "Unpolarized capacitor, small symbol"
+			(at 73.66 68.58 0)
+			(effects
+				(font
+					(size 1.27 1.27)
+				)
+				(hide yes)
+			)
+		)
+		(pin "1"
+		)
+		(pin "2"
+		)
+		(instances
+			(project "main-board"
+				(path "/c621b5fd-2ef7-4a67-960d-0ffc72b1245a/a4a3f1ff-d673-4de4-9dae-3d1051c84f77"
+					(reference "C49")
+					(unit 1)
+				)
+			)
+		)
+	)
+	(symbol
+		(lib_id "symbol-library-capacitors:CC0402KRX7R6BB104")
 		(at 87.63 68.58 0)
 		(unit 1)
@@
 			)
 		)
-		(property "Footprint" ""
+		(property "Footprint" "Capacitor_SMD:C_0402_1005Metric"
 			(at 87.63 68.58 0)
 			(effects
@@
 			)
 		)
+		(pin "1"
+		)
 		(pin "2"
 		)
-		(pin "1"
-		)
 		(instances
 			(project "main-board"
 				(path "/c621b5fd-2ef7-4a67-960d-0ffc72b1245a/a4a3f1ff-d673-4de4-9dae-3d1051c84f77"
 					(reference "C50")
+					(unit 1)
+				)
+			)
+		)
+	)
+	(symbol
+		(lib_id "symbol-library-capacitors:CC0402MRX5R6BB475")
+		(at 101.6 68.58 0)
+		(unit 1)
+		(exclude_from_sim no)
+		(in_bom yes)
+		(on_board yes)
+		(dnp no)
+		(fields_autoplaced yes)
+		(property "Reference" "C51"
+			(at 104.14 67.3162 0)
+			(effects
+				(font
+					(size 1.27 1.27)
+				)
+				(justify left)
+			)
+		)
+		(property "Value" "4.7uF 10V"
+			(at 104.14 69.8562 0)
+			(effects
+				(font
+					(size 1.27 1.27)
+				)
+				(justify left)
+			)
+		)
+		(property "Footprint" "Capacitor_SMD:C_0402_1005Metric"
+			(at 101.6 68.58 0)
+			(effects
+				(font
+					(size 1.27 1.27)
+				)
+				(hide yes)
+			)
+		)
+		(property "Datasheet" "~"
+			(at 101.6 68.58 0)
+			(effects
+				(font
+					(size 1.27 1.27)
+				)
+				(hide yes)
+			)
+		)
+		(property "Description" "Unpolarized capacitor, small symbol"
+			(at 101.6 68.58 0)
+			(effects
+				(font
+					(size 1.27 1.27)
+				)
+				(hide yes)
+			)
+		)
+		(pin "1"
+		)
+		(pin "2"
+		)
+		(instances
+			(project "main-board"
+				(path "/c621b5fd-2ef7-4a67-960d-0ffc72b1245a/a4a3f1ff-d673-4de4-9dae-3d1051c84f77"
+					(reference "C51")
 					(unit 1)
 				)
@@
 		(dnp no)
 		(fields_autoplaced yes)
-		(property "Reference" "#PWR083"
+		(property "Reference" "#PWR082"
 			(at 73.66 78.74 0)
 			(effects
@@
 			(project "main-board"
 				(path "/c621b5fd-2ef7-4a67-960d-0ffc72b1245a/a4a3f1ff-d673-4de4-9dae-3d1051c84f77"
-					(reference "#PWR083")
-					(unit 1)
-				)
-			)
-		)
-	)
-	(symbol
-		(lib_id "Device:C_Small")
-		(at 73.66 68.58 0)
-		(unit 1)
-		(exclude_from_sim no)
-		(in_bom yes)
-		(on_board yes)
-		(dnp no)
-		(fields_autoplaced yes)
-		(property "Reference" "C49"
-			(at 76.2 67.3162 0)
-			(effects
-				(font
-					(size 1.27 1.27)
-				)
-				(justify left)
-			)
-		)
-		(property "Value" "100nF 10V"
-			(at 76.2 69.8562 0)
-			(effects
-				(font
-					(size 1.27 1.27)
-				)
-				(justify left)
-			)
-		)
-		(property "Footprint" ""
-			(at 73.66 68.58 0)
-			(effects
-				(font
-					(size 1.27 1.27)
-				)
-				(hide yes)
-			)
-		)
-		(property "Datasheet" "~"
-			(at 73.66 68.58 0)
-			(effects
-				(font
-					(size 1.27 1.27)
-				)
-				(hide yes)
-			)
-		)
-		(property "Description" "Unpolarized capacitor, small symbol"
-			(at 73.66 68.58 0)
-			(effects
-				(font
-					(size 1.27 1.27)
-				)
-				(hide yes)
-			)
-		)
-		(pin "2"
-		)
-		(pin "1"
-		)
-		(instances
-			(project ""
-				(path "/c621b5fd-2ef7-4a67-960d-0ffc72b1245a/a4a3f1ff-d673-4de4-9dae-3d1051c84f77"
-					(reference "C49")
-					(unit 1)
-				)
-			)
-		)
-	)
-	(symbol
-		(lib_id "Device:C_Small")
-		(at 115.57 68.58 0)
-		(unit 1)
-		(exclude_from_sim no)
-		(in_bom yes)
-		(on_board yes)
-		(dnp no)
-		(fields_autoplaced yes)
-		(property "Reference" "C52"
-			(at 118.11 67.3162 0)
-			(effects
-				(font
-					(size 1.27 1.27)
-				)
-				(justify left)
-			)
-		)
-		(property "Value" "4.7uF 10V"
-			(at 118.11 69.8562 0)
-			(effects
-				(font
-					(size 1.27 1.27)
-				)
-				(justify left)
-			)
-		)
-		(property "Footprint" ""
-			(at 115.57 68.58 0)
-			(effects
-				(font
-					(size 1.27 1.27)
-				)
-				(hide yes)
-			)
-		)
-		(property "Datasheet" "~"
-			(at 115.57 68.58 0)
-			(effects
-				(font
-					(size 1.27 1.27)
-				)
-				(hide yes)
-			)
-		)
-		(property "Description" "Unpolarized capacitor, small symbol"
-			(at 115.57 68.58 0)
-			(effects
-				(font
-					(size 1.27 1.27)
-				)
-				(hide yes)
-			)
-		)
-		(pin "2"
-		)
-		(pin "1"
-		)
-		(instances
-			(project "main-board"
-				(path "/c621b5fd-2ef7-4a67-960d-0ffc72b1245a/a4a3f1ff-d673-4de4-9dae-3d1051c84f77"
-					(reference "C52")
+					(reference "#PWR082")
 					(unit 1)
 				)
@@
 		(dnp no)
 		(fields_autoplaced yes)
-		(property "Reference" "#PWR084"
+		(property "Reference" "#PWR083"
 			(at 189.23 143.51 0)
 			(effects
@@
 			(project ""
 				(path "/c621b5fd-2ef7-4a67-960d-0ffc72b1245a/a4a3f1ff-d673-4de4-9dae-3d1051c84f77"
-					(reference "#PWR084")
-					(unit 1)
-				)
+					(reference "#PWR083")
+					(unit 1)
+				)

Commit message: Replace placeholder resistors
Parts:
- removed R40: 10K, symbol Device:R_Small_US
- added R36: 10K, Resistor_SMD:R_0402_1005Metric, symbol symbol-library-resistors:RC0402JR-0710KL
Connections:
- net 1V8: now also R36.1
- net RAM_HEXASPI.CS_N: now also R36.2
Changed lines of the file:
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@@
-	)
-	(symbol
-		(lib_id "Device:R_Small_US")
-		(at 138.43 71.12 0)
-		(unit 1)
-		(exclude_from_sim no)
-		(in_bom yes)
-		(on_board yes)
-		(dnp no)
-		(fields_autoplaced yes)
-		(property "Reference" "R40"
-			(at 140.97 69.8499 0)
-			(effects
-				(font
-					(size 1.27 1.27)
-				)
-				(justify left)
-			)
-		)
-		(property "Value" "10K"
-			(at 140.97 72.3899 0)
-			(effects
-				(font
-					(size 1.27 1.27)
-				)
-				(justify left)
-			)
-		)
-		(property "Footprint" ""
-			(at 138.43 71.12 0)
-			(effects
-				(font
-					(size 1.27 1.27)
-				)
-				(hide yes)
-			)
-		)
-		(property "Datasheet" "~"
-			(at 138.43 71.12 0)
-			(effects
-				(font
-					(size 1.27 1.27)
-				)
-				(hide yes)
-			)
-		)
-		(property "Description" "Resistor, small US symbol"
-			(at 138.43 71.12 0)
-			(effects
-				(font
-					(size 1.27 1.27)
-				)
-				(hide yes)
-			)
-		)
-		(pin "1"
-		)
-		(pin "2"
-		)
-		(instances
-			(project ""
-				(path "/c621b5fd-2ef7-4a67-960d-0ffc72b1245a/a4a3f1ff-d673-4de4-9dae-3d1051c84f77"
-					(reference "R40")
-					(unit 1)
-				)
-			)
-		)
 	)
 	(symbol
@@
 					(unit 1)
 				)
+			)
+		)
+	)
+	(symbol
+		(lib_id "symbol-library-resistors:RC0402JR-0710KL")
+		(at 138.43 71.12 0)
+		(unit 1)
+		(exclude_from_sim no)
+		(in_bom yes)
+		(on_board yes)
+		(dnp no)
+		(fields_autoplaced yes)
+		(property "Reference" "R36"
+			(at 140.97 69.8499 0)
+			(effects
+				(font
+					(size 1.27 1.27)
+				)
+				(justify left)
+			)
+		)
+		(property "Value" "10K"
+			(at 140.97 72.3899 0)
+			(effects
+				(font
+					(size 1.27 1.27)
+				)
+				(justify left)
+			)
+		)
+		(property "Footprint" "Resistor_SMD:R_0402_1005Metric"
+			(at 138.43 71.12 0)
+			(effects
+				(font
+					(size 1.27 1.27)
+				)
+				(hide yes)
+			)
+		)
+		(property "Datasheet" "~"
+			(at 138.43 71.12 0)
+			(effects
+				(font
+					(size 1.27 1.27)
+				)
+				(hide yes)
+			)
+		)
+		(property "Description" "Resistor, small US symbol"
+			(at 138.43 71.12 0)
+			(effects
+				(font
+					(size 1.27 1.27)
+				)
+				(hide yes)
+			)
+		)
+		(pin "1"
+		)
+		(pin "2"
+		)
+		(instances
+			(project "main-board"
+				(path "/c621b5fd-2ef7-4a67-960d-0ffc72b1245a/a4a3f1ff-d673-4de4-9dae-3d1051c84f77"
+					(reference "R36")
+					(unit 1)
+				)

Commit message: Add footprints
- Inductors
- Switches
- Buttons
Parts:
- renumbered R36 to R40
Changed lines of the file:
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@@
 		(dnp no)
 		(fields_autoplaced yes)
-		(property "Reference" "R36"
+		(property "Reference" "R40"
 			(at 140.97 69.8499 0)
 			(effects
@@
 			(project "main-board"
 				(path "/c621b5fd-2ef7-4a67-960d-0ffc72b1245a/a4a3f1ff-d673-4de4-9dae-3d1051c84f77"
-					(reference "R36")
+					(reference "R40")
 					(unit 1)
 				)
