File: projects/main-board/lcd.kicad_sch (KiCad schematic)
At the start: 10 parts, among them J6 NHD-4.3-480272EF-ASXP (Molex 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, U10 AP5725WG-7

Commit message: Rough PCB component grouping and layout
Changed lines of the file:
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@@
+	)
+	(junction
+		(at 121.92 41.91)
+		(diameter 0)
+		(color 0 0 0 0)
 	)
 	(junction
@@
 	)
 	(junction
-		(at 110.49 41.91)
-		(diameter 0)
-		(color 0 0 0 0)
-	)
-	(junction
 		(at 260.35 135.89)
 		(diameter 0)
@@
 		)
 	)
-	(wire
-		(pts
-			(xy 110.49 41.91) (xy 121.92 41.91)
-		)
-		(stroke
-			(width 0)
-			(type default)
-		)
-	)
 	(bus
 		(pts
@@
 	(wire
 		(pts
-			(xy 91.44 41.91) (xy 110.49 41.91)
+			(xy 91.44 41.91) (xy 121.92 41.91)
 		)
 		(stroke
@@
 	(symbol
 		(lib_id "power:VCC")
-		(at 110.49 41.91 0)
+		(at 121.92 41.91 0)
 		(unit 1)
 		(exclude_from_sim no)
@@
 		(fields_autoplaced yes)
 		(property "Reference" "#PWR0127"
-			(at 110.49 45.72 0)
+			(at 121.92 45.72 0)
 			(effects
 				(font
@@
 		)
 		(property "Value" "BACKLIGHT_P"
-			(at 110.49 36.83 0)
+			(at 121.92 36.83 0)
 			(effects
 				(font
@@
 		)
 		(property "Footprint" ""
-			(at 110.49 41.91 0)
+			(at 121.92 41.91 0)
 			(effects
 				(font
@@
 		)
 		(property "Datasheet" ""
-			(at 110.49 41.91 0)
+			(at 121.92 41.91 0)
 			(effects
 				(font
@@
 		)
 		(property "Description" "Power symbol creates a global label with name \"VCC\""
-			(at 110.49 41.91 0)
-			(effects
-				(font
+			(at 121.92 41.91 0)
+			(effects
+				(font

Commit message: WIP splitting main board into 3
Other:
- moved on the sheet: C87, C88, C89, C90, D1, J6, L6, R55, R56, U10
