File: projects/main-board/usb-switch.kicad_sch (KiCad schematic)
At the start: 2 parts

Commit message: Updated schematics with new symbols
Parts:
- removed U5: ~, symbol symbol-library:TS3USB221ARSER
- added U4: TS3USB221ARSER, footprint-library:TS3USB221ARSER, symbol symbol-library:TS3USB221ARSER
Connections:
- net 3V3: now also U4.10 (VCC)
- net GND: now also U4.5 (GND), U4.6 (OE_N)
- net SELECT_PORT_2: now also U4.9 (S)
- net USB_DOWN_1.DN: now also U4.2 (1D-)
- net USB_DOWN_1.DP: now also U4.1 (1D+)
- net USB_DOWN_2.DN: now also U4.4 (2D-)
- net USB_DOWN_2.DP: now also U4.3 (2D+)
- net USB_UP.DN: now also U4.7 (D-)
- net USB_UP.DP: now also U4.8 (D+)
Changed lines of the file:
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@@
+	)
+	(symbol
+		(lib_name "TS3USB221ARSER_1")
+		(lib_id "symbol-library:TS3USB221ARSER")
+		(at 138.43 82.55 0)
+		(unit 1)
+		(exclude_from_sim no)
+		(in_bom yes)
+		(on_board yes)
+		(dnp no)
+		(fields_autoplaced yes)
+		(property "Reference" "U4"
+			(at 151.765 77.47 0)
+			(effects
+				(font
+					(size 1.27 1.27)
+				)
+			)
+		)
+		(property "Value" "TS3USB221ARSER"
+			(at 151.765 80.01 0)
+			(effects
+				(font
+					(size 1.27 1.27)
+				)
+			)
+		)
+		(property "Footprint" "footprint-library:TS3USB221ARSER"
+			(at 152.654 107.188 0)
+			(effects
+				(font
+					(size 1.27 1.27)
+				)
+				(hide yes)
+			)
+		)
+		(property "Datasheet" ""
+			(at 138.43 82.55 0)
+			(effects
+				(font
+					(size 1.27 1.27)
+				)
+				(hide yes)
+			)
+		)
+		(property "Description" ""
+			(at 138.43 82.55 0)
+			(effects
+				(font
+					(size 1.27 1.27)
+				)
+				(hide yes)
+			)
+		)
+		(pin "6"
+		)
+		(pin "9"
+		)
+		(pin "8"
+		)
+		(pin "7"
+		)
+		(pin "1"
+		)
+		(pin "2"
+		)
+		(pin "3"
+		)
+		(pin "4"
+		)
+		(pin "5"
+		)
+		(pin "10"
+		)
+		(instances
+			(project ""
+				(path "/c621b5fd-2ef7-4a67-960d-0ffc72b1245a/a8fc3290-2c1b-45f6-84c7-bf573b237fec"
+					(reference "U4")
+					(unit 1)
+				)
+			)
+		)
 	)
 	(symbol
@@
 					(unit 1)
 				)
-			)
-		)
-	)
-	(symbol
-		(lib_id "symbol-library:TS3USB221ARSER")
-		(at 138.43 82.55 0)
-		(unit 1)
-		(exclude_from_sim no)
-		(in_bom yes)
-		(on_board yes)
-		(dnp no)
-		(property "Reference" "U5"
-			(at 139.7 81.28 0)
-			(effects
-				(font
-					(size 1.27 1.27)
-				)
-			)
-		)
-		(property "Value" "~"
-			(at 142.748 81.28 0)
-			(effects
-				(font
-					(size 1.27 1.27)
-				)
-			)
-		)
-		(property "Footprint" ""
-			(at 138.43 82.55 0)
-			(effects
-				(font
-					(size 1.27 1.27)
-				)
-				(hide yes)
-			)
-		)
-		(property "Datasheet" ""
-			(at 138.43 82.55 0)
-			(effects
-				(font
-					(size 1.27 1.27)
-				)
-				(hide yes)
-			)
-		)
-		(property "Description" ""
-			(at 138.43 82.55 0)
-			(effects
-				(font
-					(size 1.27 1.27)
-				)
-				(hide yes)
-			)
-		)
-		(pin "6"
-		)
-		(pin "9"
-		)
-		(pin "10"
-		)
-		(pin "1"
-		)
-		(pin "2"
-		)
-		(pin "3"
-		)
-		(pin "4"
-		)
-		(pin "5"
-		)
-		(pin "8"
-		)
-		(pin "7"
-		)
-		(instances
-			(project ""
-				(path "/c621b5fd-2ef7-4a67-960d-0ffc72b1245a/a8fc3290-2c1b-45f6-84c7-bf573b237fec"
-					(reference "U5")
-					(unit 1)
-				)

Commit message: Re-annotate schematics.
Parts:
- renumbered C59 to C74, U4 to U8
Changed lines of the file:
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@@
 		(dnp no)
 		(fields_autoplaced yes)
-		(property "Reference" "#PWR082"
+		(property "Reference" "#PWR0114"
 			(at 168.91 110.49 0)
 			(effects
@@
 			(project ""
 				(path "/c621b5fd-2ef7-4a67-960d-0ffc72b1245a/a8fc3290-2c1b-45f6-84c7-bf573b237fec"
-					(reference "#PWR082")
+					(reference "#PWR0114")
 					(unit 1)
 				)
@@
 		(dnp no)
 		(fields_autoplaced yes)
-		(property "Reference" "U4"
+		(property "Reference" "U8"
 			(at 151.765 77.47 0)
 			(effects
@@
 			(project ""
 				(path "/c621b5fd-2ef7-4a67-960d-0ffc72b1245a/a8fc3290-2c1b-45f6-84c7-bf573b237fec"
-					(reference "U4")
+					(reference "U8")
 					(unit 1)
 				)
@@
 		(dnp no)
 		(fields_autoplaced yes)
-		(property "Reference" "#PWR081"
+		(property "Reference" "#PWR0112"
 			(at 92.71 87.63 0)
 			(effects
@@
 			(project ""
 				(path "/c621b5fd-2ef7-4a67-960d-0ffc72b1245a/a8fc3290-2c1b-45f6-84c7-bf573b237fec"
-					(reference "#PWR081")
+					(reference "#PWR0112")
 					(unit 1)
 				)
@@
 		(dnp no)
 		(fields_autoplaced yes)
-		(property "Reference" "C59"
+		(property "Reference" "C74"
 			(at 95.25 87.6362 0)
 			(effects
@@
 			(project ""
 				(path "/c621b5fd-2ef7-4a67-960d-0ffc72b1245a/a8fc3290-2c1b-45f6-84c7-bf573b237fec"
-					(reference "C59")
+					(reference "C74")
 					(unit 1)
 				)
@@
 		(dnp no)
 		(fields_autoplaced yes)
-		(property "Reference" "#PWR083"
+		(property "Reference" "#PWR0113"
 			(at 92.71 99.06 0)
 			(effects
@@
 			(project "main-board"
 				(path "/c621b5fd-2ef7-4a67-960d-0ffc72b1245a/a8fc3290-2c1b-45f6-84c7-bf573b237fec"
-					(reference "#PWR083")
-					(unit 1)
-				)
+					(reference "#PWR0113")
+					(unit 1)
+				)

Commit message: Normalise capacitors
- Add capacitor parts to library.
- Replace all placeholder capacitors
  with the actual part numbers.
Parts:
- removed C74: 100nF 10V, symbol Device:C_Small
- added C74: 100nF 10V, Capacitor_SMD:C_0402_1005Metric, symbol symbol-library-capacitors:CC0402KRX7R6BB104
Connections:
- net 3V3: now also C74.1
- net GND: now also C74.2
Changed lines of the file:
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@@
 	(paper "A4")
 	(junction
-		(at 92.71 85.09)
+		(at 92.71 91.44)
 		(diameter 0)
 		(color 0 0 0 0)
 	)
 	(junction
-		(at 92.71 91.44)
+		(at 92.71 85.09)
 		(diameter 0)
 		(color 0 0 0 0)
@@
 		(dnp no)
 		(fields_autoplaced yes)
-		(property "Reference" "#PWR0114"
+		(property "Reference" "#PWR0113"
 			(at 168.91 110.49 0)
 			(effects
@@
 			(project ""
 				(path "/c621b5fd-2ef7-4a67-960d-0ffc72b1245a/a8fc3290-2c1b-45f6-84c7-bf573b237fec"
-					(reference "#PWR0114")
+					(reference "#PWR0113")
 					(unit 1)
 				)
@@
 		(dnp no)
 		(fields_autoplaced yes)
-		(property "Reference" "#PWR0112"
+		(property "Reference" "#PWR0111"
 			(at 92.71 87.63 0)
 			(effects
@@
 			(project ""
 				(path "/c621b5fd-2ef7-4a67-960d-0ffc72b1245a/a8fc3290-2c1b-45f6-84c7-bf573b237fec"
+					(reference "#PWR0111")
+					(unit 1)
+				)
+			)
+		)
+	)
+	(symbol
+		(lib_id "power:GND")
+		(at 92.71 92.71 0)
+		(unit 1)
+		(exclude_from_sim no)
+		(in_bom yes)
+		(on_board yes)
+		(dnp no)
+		(fields_autoplaced yes)
+		(property "Reference" "#PWR0112"
+			(at 92.71 99.06 0)
+			(effects
+				(font
+					(size 1.27 1.27)
+				)
+				(hide yes)
+			)
+		)
+		(property "Value" "GND"
+			(at 92.71 97.79 0)
+			(effects
+				(font
+					(size 1.27 1.27)
+				)
+			)
+		)
+		(property "Footprint" ""
+			(at 92.71 92.71 0)
+			(effects
+				(font
+					(size 1.27 1.27)
+				)
+				(hide yes)
+			)
+		)
+		(property "Datasheet" ""
+			(at 92.71 92.71 0)
+			(effects
+				(font
+					(size 1.27 1.27)
+				)
+				(hide yes)
+			)
+		)
+		(property "Description" "Power symbol creates a global label with name \"GND\" , ground"
+			(at 92.71 92.71 0)
+			(effects
+				(font
+					(size 1.27 1.27)
+				)
+				(hide yes)
+			)
+		)
+		(pin "1"
+		)
+		(instances
+			(project "main-board"
+				(path "/c621b5fd-2ef7-4a67-960d-0ffc72b1245a/a8fc3290-2c1b-45f6-84c7-bf573b237fec"
 					(reference "#PWR0112")
 					(unit 1)
@@
 	)
 	(symbol
-		(lib_id "Device:C_Small")
+		(lib_id "symbol-library-capacitors:CC0402KRX7R6BB104")
 		(at 92.71 88.9 0)
 		(unit 1)
@@
 			)
 		)
-		(property "Footprint" ""
+		(property "Footprint" "Capacitor_SMD:C_0402_1005Metric"
 			(at 92.71 88.9 0)
 			(effects
@@
 			)
 		)
+		(pin "1"
+		)
 		(pin "2"
 		)
-		(pin "1"
-		)
 		(instances
-			(project ""
+			(project "main-board"
 				(path "/c621b5fd-2ef7-4a67-960d-0ffc72b1245a/a8fc3290-2c1b-45f6-84c7-bf573b237fec"
 					(reference "C74")
 					(unit 1)
 				)
-			)
-		)
-	)
-	(symbol
-		(lib_id "power:GND")
-		(at 92.71 92.71 0)
-		(unit 1)
-		(exclude_from_sim no)
-		(in_bom yes)
-		(on_board yes)
-		(dnp no)
-		(fields_autoplaced yes)
-		(property "Reference" "#PWR0113"
-			(at 92.71 99.06 0)
-			(effects
-				(font
-					(size 1.27 1.27)
-				)
-				(hide yes)
-			)
-		)
-		(property "Value" "GND"
-			(at 92.71 97.79 0)
-			(effects
-				(font
-					(size 1.27 1.27)
-				)
-			)
-		)
-		(property "Footprint" ""
-			(at 92.71 92.71 0)
-			(effects
-				(font
-					(size 1.27 1.27)
-				)
-				(hide yes)
-			)
-		)
-		(property "Datasheet" ""
-			(at 92.71 92.71 0)
-			(effects
-				(font
-					(size 1.27 1.27)
-				)
-				(hide yes)
-			)
-		)
-		(property "Description" "Power symbol creates a global label with name \"GND\" , ground"
-			(at 92.71 92.71 0)
-			(effects
-				(font
-					(size 1.27 1.27)
-				)
-				(hide yes)
-			)
-		)
-		(pin "1"
-		)
-		(instances
-			(project "main-board"
-				(path "/c621b5fd-2ef7-4a67-960d-0ffc72b1245a/a8fc3290-2c1b-45f6-84c7-bf573b237fec"
-					(reference "#PWR0113")
-					(unit 1)
-				)

Commit message: WIP splitting main board into 3
Changed lines of the file:
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@@
 		(color 0 0 0 0)
 	)
-	(bus_entry
-		(at 187.96 96.52)
-		(size 2.54 2.54)
-		(stroke
-			(width 0)
-			(type default)
-		)
-	)
-	(bus_entry
-		(at 119.38 102.87)
-		(size -2.54 2.54)
-		(stroke
-			(width 0)
-			(type default)
-		)
-	)
-	(bus_entry
-		(at 187.96 87.63)
-		(size 2.54 2.54)
-		(stroke
-			(width 0)
-			(type default)
-		)
-	)
-	(bus_entry
-		(at 187.96 93.98)
-		(size 2.54 2.54)
-		(stroke
-			(width 0)
-			(type default)
-		)
-	)
-	(bus_entry
-		(at 187.96 85.09)
-		(size 2.54 2.54)
-		(stroke
-			(width 0)
-			(type default)
-		)
-	)
-	(bus_entry
-		(at 119.38 100.33)
-		(size -2.54 2.54)
-		(stroke
-			(width 0)
-			(type default)
-		)
-	)
 	(bus
 		(pts
-			(xy 190.5 99.06) (xy 213.36 99.06)
+			(xy 128.27 55.88) (xy 105.41 55.88)
 		)
 		(stroke
@@
 	(bus
 		(pts
-			(xy 99.06 105.41) (xy 116.84 105.41)
+			(xy 105.41 48.26) (xy 123.19 48.26)
 		)
 		(stroke
@@
 	(bus
 		(pts
-			(xy 190.5 90.17) (xy 213.36 90.17)
-		)
-		(stroke
-			(width 0)
-			(type default)
-		)
-	)
-	(bus
-		(pts
-			(xy 190.5 96.52) (xy 190.5 99.06)
+			(xy 128.27 52.07) (xy 105.41 52.07)
 		)
 		(stroke
@@
 		)
 	)
-	(bus
-		(pts
-			(xy 116.84 102.87) (xy 116.84 105.41)
-		)
-		(stroke
-			(width 0)
-			(type default)
-		)
-	)
 	(wire
 		(pts
 			(xy 167.64 102.87) (xy 168.91 102.87)
-		)
-		(stroke
-			(width 0)
-			(type default)
-		)
-	)
-	(bus
-		(pts
-			(xy 190.5 87.63) (xy 190.5 90.17)
 		)
 		(stroke
@@
 	)
 	(label "USB_DOWN_2{DP DN}"
-		(at 193.04 99.06 0)
-		(effects
-			(font
-				(size 1.27 1.27)
-			)
-			(justify left bottom)
+		(at 125.73 55.88 180)
+		(effects
+			(font
+				(size 1.27 1.27)
+			)
+			(justify right bottom)
 		)
 	)
 	(label "USB_DOWN_1{DP DN}"
-		(at 193.04 90.17 0)
-		(effects
-			(font
-				(size 1.27 1.27)
-			)
-			(justify left bottom)
+		(at 125.73 52.07 180)
+		(effects
+			(font
+				(size 1.27 1.27)
+			)
+			(justify right bottom)
 		)
 	)
@@
 	)
 	(label "USB_UP{DP DN}"
-		(at 101.6 105.41 0)
+		(at 107.95 48.26 0)
 		(effects
 			(font
@@
 	(hierarchical_label "USB_DOWN_1"
 		(shape bidirectional)
-		(at 213.36 90.17 0)
-		(effects
-			(font
-				(size 1.27 1.27)
-			)
-			(justify left)
+		(at 105.41 52.07 180)
+		(effects
+			(font
+				(size 1.27 1.27)
+			)
+			(justify right)
 		)
 	)
@@
 	(hierarchical_label "USB_UP"
 		(shape bidirectional)
-		(at 99.06 105.41 180)
+		(at 105.41 48.26 180)
 		(effects
 			(font
@@
 	(hierarchical_label "USB_DOWN_2"
 		(shape bidirectional)
-		(at 213.36 99.06 0)
-		(effects
-			(font
-				(size 1.27 1.27)
-			)
-			(justify left)
-		)
-	)
+		(at 105.41 55.88 180)
+		(effects
+			(font
+				(size 1.27 1.27)
+			)
+			(justify right)
+		)
+	)
