File: projects/main-board/controllers.kicad_sch (KiCad schematic)
At the start: 2 parts, among them J8 5051101292, J9 5051101292

Commit message: Fix wrong net name on left audio
Connections:
- net LEFT_MOTOR_N renamed LEFT_MOTOR.N
Changed lines of the file:
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@@
 		)
 	)
-	(label "LEFT_MOTOR_N"
+	(label "LEFT_MOTOR.N"
 		(at 106.68 109.22 0)
 		(effects
